Commit message: pretty much functioning!

File: rosws/src/rover_description/urdf/rover.xacro.urdf (robot description, URDF)
Before this commit: robot rover, 1 links, 0 joints
Links:
- link base_link: mass 2.0 -> 1.0

File: rosws/src/rover_description/urdf/sensors.xacro (robot description, xacro)
@@ -64,5 +64,5 @@
         <inertial>
             <inertia ixx="0.000604166666667" ixy="0" ixz="0" iyy="0.000166666666667" iyz="0" izz="0.000604166666667"/>
-            <mass value="0.1"/>
+            <mass value="0.05"/>
         </inertial>
         <visual>
@@ -78,17 +78,28 @@
     </link>
     <joint name="base_to_imu_link" type="fixed">
-        <parent link="base_link" />
-        <child link="imu_link" />
-        <origin xyz="0 0 0.125" />
+        <parent link="base_link"/>
+        <child link="imu_link"/>
+        <origin xyz="0 0 0.125"/>
     </joint>
-    <gazebo>
-        <plugin name="imu_plugin" filename="libhector_gazebo_ros_imu.so">
-            <alwaysOn>true</alwaysOn>
-            <bodyName>imu_link</bodyName>
-            <topicName>/imu/data</topicName>
-            <serviceName>/imu/service</serviceName>
-            <gaussianNoise>0.1</gaussianNoise>
-            <updateRate>20.0</updateRate>
-        </plugin>
+    <gazebo reference="imu_link">
+        <gravity>true</gravity>
+        <sensor name="imu_sensor" type="imu">
+            <always_on>true</always_on>
+            <update_rate>100</update_rate>
+            <visualize>true</visualize>
+            <topic>__default_topic__</topic>
+            <plugin name="imu_plugin" filename="libgazebo_ros_imu_sensor.so">
+                <alwaysOn>true</alwaysOn>
+                <bodyName>imu_link</bodyName>
+                <topicName>/imu/data</topicName>
+                <serviceName>/imu/service</serviceName>
+                <gaussianNoise>0.05</gaussianNoise>
+                <updateRateHZ>20.0</updateRateHZ>
+                <xyzOffset>0 0 0</xyzOffset>
+                <rpyOffset>0 0 0</rpyOffset>
+                <frameName>imu_link</frameName>
+            </plugin>
+            <pose>0 0 0 0 0 0</pose> <!-- todo: make sure this is right -->
+        </sensor>
     </gazebo>
 </robot>

File: rosws/src/rover_description/urdf/wheel.xacro (robot description, xacro)
@@ -28,5 +28,5 @@
         <link name="wheel_${suffix}">
             <inertial>
-                <mass value="1" />
+                <mass value="0.25" />
                 <inertia ixx="0.00333333333333" ixy="0" ixz="0" iyy="0.005" iyz="0" izz="0.00333333333333" />
             </inertial>
@@ -60,5 +60,5 @@
                     <friction>
                         <torsional>
-                            <coefficient>0.5</coefficient>
+                            <coefficient>0.6</coefficient>
                             <use_patch_radius>true</use_patch_radius>
                             <patch_radius>0.1</patch_radius>
