Commit message: working gazebo config w/ simple rover

File: rosws/src/rover_description/urdf/wheel.xacro (robot description, xacro)
@@ -1,4 +1,5 @@
+<?xml version="1.0" ?>
 <robot xmlns:xacro="http://www.ros.org/wiki/xacro">
-    <xacro:macro name="wheel_leg" params="suffix attach">
+    <xacro:macro name="wheel" params="suffix attach side">
         <link name="wheel_leg_${suffix}">
             <inertial>
@@ -20,5 +21,5 @@
             </collision>
         </link>
-        <joint name="base_leg_${suffix}" type="fixed">
+        <joint name="base_to_leg_${suffix}" type="fixed">
             <origin xyz="${attach}" rpy="0 0 0" />
             <parent link="base_link" />
@@ -31,7 +32,26 @@
             </inertial>
             <visual>
-                <origin
+                <origin xyz="0 0 0" rpy="1.5708 0 0" />
+                <material name="White" />
+                <geometry>
+                    <cylinder radius="0.1" length="0.1" />
+                </geometry>
             </visual>
+            <collision>
+                <origin xyz="0 0 0" rpy="1.5708 0 0" />
+                <geometry>
+                    <cylinder radius="0.1" length="0.1" />
+                </geometry>
+            </collision>
         </link>
+        <joint name="leg_to_wheel_${suffix}" type="continuous">
+            <origin xyz="0 ${side * 0.1} -0.3" rpy="0 0 0" />
+            <parent link="wheel_leg_${suffix}" />
+            <child link="wheel_${suffix}" />
+            <axis xyz="0 1 0" />
+        </joint>
+        <gazebo reference="wheel_leg_${suffix}">
+            <material>Gazebo/Red</material>
+        </gazebo>
     </xacro:macro>
 </robot>

Commit message: add more stuff to make auton easier

File: rosws/src/rover_description/urdf/wheel.xacro (robot description, xacro)
@@ -50,5 +50,5 @@
             <child link="wheel_${suffix}" />
             <axis xyz="0 1 0" />
-            <dynamics damping="0.015" friction="0.02" />
+            <!-- dynamics damping="0.015" friction="0.02" / -->
         </joint>
         <gazebo reference="wheel_leg_${suffix}">

Commit message: yippe yooooooo!
in other words, it functions now

(cherry picked from commit a7708cd)

File: rosws/src/rover_description/urdf/wheel.xacro (robot description, xacro)
@@ -50,5 +50,5 @@
             <child link="wheel_${suffix}" />
             <axis xyz="0 1 0" />
-            <!-- dynamics damping="0.015" friction="0.02" / -->
+            <dynamics damping="0.015" friction="0.02" />
         </joint>
         <gazebo reference="wheel_leg_${suffix}">
@@ -56,6 +56,15 @@
         </gazebo>
         <gazebo reference="wheel_${suffix}">
-            <mu1 value="0.8" />
-            <mu2 value="0.8" />
+            <collision name="wheel_${suffix}_collision">
+                <surface>
+                    <friction>
+                        <torsional>
+                            <coefficient>0.5</coefficient>
+                            <use_patch_radius>true</use_patch_radius>
+                            <patch_radius>0.1</patch_radius>
+                        </torsional>
+                    </friction>
+                </surface>
+            </collision>
         </gazebo>
         <transmission name="wheel_transmission_${suffix}">

Commit message: Wheel friction fix (#9)
* Remove simple_drive.launch

It was just a poop anyways

* yippe yooooooo!

in other words, it functions now

File: rosws/src/rover_description/urdf/wheel.xacro (robot description, xacro)
@@ -56,8 +56,15 @@
         </gazebo>
         <gazebo reference="wheel_${suffix}">
-            <kp value="100000" />
-            <kd value="1.0" />
-            <mu1 value="0.5" />
-            <mu2 value="0.5" />
+            <collision name="wheel_${suffix}_collision">
+                <surface>
+                    <friction>
+                        <torsional>
+                            <coefficient>0.5</coefficient>
+                            <use_patch_radius>true</use_patch_radius>
+                            <patch_radius>0.1</patch_radius>
+                        </torsional>
+                    </friction>
+                </surface>
+            </collision>
         </gazebo>
         <transmission name="wheel_transmission_${suffix}">

Commit message: holy fuck

File: rosws/src/rover_description/urdf/wheel.xacro (robot description, xacro)
@@ -50,5 +50,5 @@
             <child link="wheel_${suffix}" />
             <axis xyz="0 1 0" />
-            <!-- dynamics damping="0.015" friction="0.02" / -->
+            <dynamics damping="0.015" friction="0.02" />
         </joint>
         <gazebo reference="wheel_leg_${suffix}">
