Commit message: holy code dump. also moveit works now and there's an arm

File: rosws/src/rover_description/urdf/arm.xacro (robot description, xacro)
@@ -1,3 +1,389 @@
 <?xml version="1.0" ?>
 <robot xmlns:xacro="http://www.ros.org/wiki/xacro">
+    <link name="arm_base">
+        <inertial>
+            <mass value="0.2"/>
+            <inertia ixx="0.000416666666667" ixy="0" ixz="0" iyy="0.000416666666667" iyz="0" izz="0.00075"/>
+        </inertial>
+        <visual>
+            <origin xyz="0 0 0.025" rpy="0 0 0"/>
+            <material name="Red"/>
+            <geometry>
+                <box size="0.15 0.15 0.05"/>
+            </geometry>
+        </visual>
+        <collision>
+            <origin xyz="0 0 0.025" rpy="0 0 0"/>
+            <geometry>
+                <box size="0.15 0.15 0.05"/>
+            </geometry>
+        </collision>
+    </link>
+    <joint name="base_to_arm_base" type="fixed">
+        <parent link="base_link"/>
+        <child link="arm_base"/>
+        <origin xyz="-0.375 0 0.25" rpy="0 0 0"/>
+    </joint>
+    <xacro:linkColor link="arm_base" mat="Gazebo/Red"/>
+    <link name="arm_post">
+        <inertial>
+            <mass value="1.5"/>
+            <inertia ixx="0.02135" ixy="0" ixz="0" iyy="0.02135" iyz="0" izz="0.0027"/>
+        </inertial>
+        <visual>
+            <origin xyz="0 0 0.2" rpy="0 0 0"/>
+            <material name="Blue"/>
+            <geometry>
+                <cylinder radius="0.06" length="0.4"/>
+            </geometry>
+        </visual>
+        <collision>
+            <origin xyz="0 0 0.2" rpy="0 0 0"/>
+            <geometry>
+                <cylinder radius="0.06" length="0.4"/>
+            </geometry>
+        </collision>
+    </link>
+    <xacro:linkColor link="arm_post" mat="Gazebo/Blue"/>
+    <joint name="arm_base_to_post" type="continuous">
+        <parent link="arm_base"/>
+        <child link="arm_post"/>
+        <origin xyz="0 0 0.05"/>
+        <axis xyz="0 0 1"/>
+    </joint>
+    <link name="arm_inner_xy">
+        <inertial>
+            <mass value="0.2"/>
+            <inertia ixx="0.00618" ixy="0" ixz="0" iyy="0.00618" iyz="0" izz="0.00036"/>
+        </inertial>
+        <visual>
+            <origin xyz="0 0 0.3" rpy="0 0 0"/>
+            <material name="Yellow"/>
+            <geometry>
+                <cylinder radius="0.06" length="0.6"/>
+            </geometry>
+        </visual>
+        <collision>
+            <origin xyz="0 0 0.3" rpy="0 0 0"/>
+            <geometry>
+                <cylinder radius="0.06" length="0.6"/>
+            </geometry>
+        </collision>
+    </link>
+    <joint name="arm_post_to_inner_xy" type="fixed">
+        <parent link="arm_post"/>
+        <child link="arm_inner_xy"/>
+        <origin xyz="0 0 0.4" rpy="0 -1.5708 0"/>
+    </joint>
+    <xacro:linkColor link="arm_inner_xy" mat="Gazebo/Yellow"/>
+    <link name="arm_outer_xy">
+        <inertial>
+            <mass value="0.2"/>
+            <inertia ixx="0.00618" ixy="0" ixz="0" iyy="0.00618" iyz="0" izz="0.00036"/>
+        </inertial>
+        <visual>
+            <origin xyz="0 0 0.3" rpy="0 0 0"/>
+            <material name="Yellow"/>
+            <geometry>
+                <cylinder radius="0.06" length="0.6"/>
+            </geometry>
+        </visual>
+        <collision>
+            <origin xyz="0 0 0.3" rpy="0 0 0"/>
+            <geometry>
+                <cylinder radius="0.06" length="0.6"/>
+            </geometry>
+        </collision>
+    </link>
+    <xacro:linkColor link="arm_outer_xy" mat="Gazebo/Yellow"/>
+    <joint name="arm_inner_to_outer_xy" type="continuous">
+        <parent link="arm_inner_xy"/>
+        <child link="arm_outer_xy"/>
+        <origin xyz="0 0 0.6" rpy="0 0 0"/>
+        <axis xyz="1 0 0"/>
+    </joint>
+    <link name="arm_slide_holder">
+        <inertial>
+            <mass value="0.15"/>
+            <inertia ixx="0.00025" ixy="0" ixz="0" iyy="0.00025" iyz="0" izz="0.00025"/>
+        </inertial>
+        <visual>
+            <origin xyz="-0.05 0 0" rpy="0 0 0"/>
+            <material name="Red"/>
+            <geometry>
+                <box size="0.1 0.1 0.1"/>
+            </geometry>
+        </visual>
+        <collision>
+            <origin xyz="0 0 0.05" rpy="0 0 0"/>
+            <geometry>
+                <box size="0.1 0.1 0.1"/>
+            </geometry>
+        </collision>
+    </link>
+    <xacro:linkColor mat="Gazebo/Red" link="arm_slide_holder"/>
+    <joint name="arm_outer_xy_to_slide_holder" type="fixed">
+        <parent link="arm_outer_xy"/>
+        <child link="arm_slide_holder"/>
+        <origin xyz="0 0 0.6" rpy="0 1.5708 0"/>
+    </joint>
+    <link name="arm_z">
+        <inertial>
+            <mass value="0.2"/>
+            <inertia ixx="0.0141233333333" ixy="0" ixz="0" iyy="0.0141233333333" iyz="0" izz="8e-05"/>
+        </inertial>
+        <visual>
+            <material name="Blue"/>
+            <origin xyz="0 0 -0.65" rpy="0 0 0"/>
+            <geometry>
+                <cylinder length="1.3" radius="0.04"/>
+            </geometry>
+        </visual>
+        <collision>
+            <origin xyz="0 0 -0.65" rpy="0 0 0"/>
+            <geometry>
+                <cylinder length="1.3" radius="0.04"/>
+            </geometry>
+        </collision>
+    </link>
+    <xacro:linkColor link="arm_z" mat="Gazebo/Blue"/>
+    <joint name="arm_z_slide" type="prismatic">
+        <parent link="arm_slide_holder"/>
+        <child link="arm_z"/>
+        <origin xyz="-0.05 0 0.65" rpy="0 0 0"/>
+        <axis xyz="0 0 1"/>
+        <limit effort="15" velocity="0.02" lower="-0.6" upper="0.6"/>
+    </joint>
+    <link name="arm_gripper_rotate_z">
+        <inertial>
+            <mass value="0.1"/>
+            <inertia ixx="4.08333333333e-05" ixy="0" ixz="0" iyy="4.08333333333e-05" iyz="0" izz="8e-05"/>
+        </inertial>
+        <visual>
+            <material name="White"/>
+            <origin xyz="0 0 -0.025" rpy="0 0 0"/>
+            <geometry>
+                <cylinder radius="0.04" length="0.05"/>
+            </geometry>
+        </visual>
+        <collision>
+            <origin xyz="0 0 -0.025" rpy="0 0 0"/>
+            <geometry>
+                <cylinder radius="0.04" length="0.05"/>
+            </geometry>
+        </collision>
+    </link>
+    <joint name="arm_gripper_rot_z" type="continuous">
+        <parent link="arm_z"/>
+        <child link="arm_gripper_rotate_z"/>
+        <origin xyz="0 0 -1.3" rpy="0 0 0"/>
+        <axis xyz="0 0 1"/>
+    </joint>
+    <link name="arm_gripper_rotate_y">
+        <inertial>
+            <mass value="0.1"/>
+            <inertia ixx="4.08333333333e-05" ixy="0" ixz="0" iyy="4.08333333333e-05" iyz="0" izz="8e-05"/>
+        </inertial>
+        <visual>
+            <material name="White"/>
+            <origin xyz="0 0 -0.025" rpy="0 0 0"/>
+            <geometry>
+                <cylinder radius="0.04" length="0.05"/>
+            </geometry>
+        </visual>
+        <collision>
+            <origin xyz="0 0 -0.025" rpy="0 0 0"/>
+            <geometry>
+                <cylinder radius="0.04" length="0.05"/>
+            </geometry>
+        </collision>
+    </link>
+    <joint name="arm_gripper_rot_y" type="revolute">
+        <parent link="arm_gripper_rotate_z"/>
+        <child link="arm_gripper_rotate_y"/>
+        <origin xyz="0 0 -0.05" rpy="0 0 0"/>
+        <axis xyz="0 1 0"/>
+        <limit effort="7" velocity="0.025" lower="-1.4" upper="1.4" />
+    </joint>
+    <link name="gripper_base">
+        <inertial>
+            <mass value="0.3" />
+            <inertia ixx="0.0019375" ixy="0" ixz="0" iyy="0.0019375" iyz="0" izz="0.003375" />
+        </inertial>
+        <visual>
+            <material name="Yellow" />
+            <origin xyz="0 0 -0.05" rpy="0 0 0" />
+            <geometry>
+                <cylinder length="0.1" radius="0.15" />
+            </geometry>
+        </visual>
+        <collision>
+            <origin xyz="0 0 -0.05" rpy="0 0 0" />
+            <geometry>
+                <cylinder length="0.1" radius="0.15" />
+            </geometry>
+        </collision>
+    </link>
+    <joint name="arm_to_gripper" type="fixed">
+        <parent link="arm_gripper_rotate_y" />
+        <child link="gripper_base" />
+        <origin xyz="0 0 -0.05" />
+    </joint>
+    <xacro:macro name="finger" params="suffix">
+        <link name="gripper_finger_lower_${suffix}">
+            <inertial>
+                <mass value="0.08" />
+                <inertia ixx="0.000158" ixy="0" ixz="0" iyy="0.000158" iyz="0" izz="1.6e-05" />
+            </inertial>
+            <visual>
+                <origin xyz="0 0 -0.05" rpy="0 0 0" />
+                <material name="White" />
+                <geometry>
+                    <cylinder radius="0.02" length="0.1" />
+                </geometry>
+            </visual>
+            <collision>
+                <origin xyz="0 0 -0.075" rpy="0 0 0" />
+                <geometry>
+                    <cylinder radius="0.02" length="0.1" />
+                </geometry>
+            </collision>
+        </link>
+        <link name="gripper_finger_upper_${suffix}">
+            <inertial>
+                <mass value="0.08" />
+                <inertia ixx="0.000158" ixy="0" ixz="0" iyy="0.000158" iyz="0" izz="1.6e-05" />
+            </inertial>
+            <visual>
+                <origin xyz="0 0 -0.05" rpy="0 0 0" />
+                <material name="White" />
+                <geometry>
+                    <cylinder radius="0.02" length="0.1" />
+                </geometry>
+            </visual>
+            <collision>
+                <origin xyz="0 0 -0.075" rpy="0 0 0" />
+                <geometry>
+                    <cylinder radius="0.02" length="0.1" />
+                </geometry>
+            </collision>
+        </link>
+        <joint name="gripper_finger_link_${suffix}" type="fixed">
+            <parent link="gripper_finger_lower_${suffix}" />
+            <child  link="gripper_finger_upper_${suffix}" />
+            <origin xyz="0 0 -0.1" rpy="0 0.55 0" />
+        </joint>
+    </xacro:macro>
+    <xacro:finger suffix="front_left" />
+    <xacro:finger suffix="front_right" />
+    <xacro:finger suffix="back_left" />
+    <xacro:finger suffix="back_right" />
+    <joint name="gripper_base_to_finger_front_left" type="revolute">
+        <parent link="gripper_base" />
+        <child link="gripper_finger_lower_front_left" />
+        <origin xyz="0.10605 -0.10605 -0.1" rpy="0 0 -0.7853" />
+        <axis xyz="0 -1 0" />
+        <limit effort="10" velocity="0.05" lower="0" upper="0.55"/>
+    </joint>
+    <joint name="gripper_base_to_finger_front_right" type="revolute">
+        <parent link="gripper_base" />
+        <child link="gripper_finger_lower_front_right" />
+        <origin xyz="0.10605 0.10605 -0.1" rpy="0 0 0.7853" />
+        <axis xyz="0 -1 0" />
+        <limit effort="10" velocity="0.05" lower="0" upper="0.55"/>
+    </joint>
+    <joint name="gripper_base_to_finger_back_left" type="revolute">
+        <parent link="gripper_base" />
+        <child link="gripper_finger_lower_back_left" />
+        <origin xyz="-0.10605 -0.10605 -0.1" rpy="0 0 -2.35619449" />
+        <axis xyz="0 -1 0" />
+        <limit effort="10" velocity="0.05" lower="0" upper="0.55"/>
+    </joint>
+    <joint name="gripper_base_to_finger_back_right" type="revolute">
+        <parent link="gripper_base" />
+        <child link="gripper_finger_lower_back_right" />
+        <origin xyz="-0.10605 0.10605 -0.1" rpy="0 0 2.35619449" />
+        <axis xyz="0 -1 0" />
+        <limit effort="10" velocity="0.05" lower="0" upper="0.55"/>
+    </joint>
+    <transmission name="arm_post_rotate_trans">
+        <type>transmission_interface/SimpleTransmission</type>
+        <joint name="arm_base_to_post">
+            <hardwareInterface>hardware_interface/VelocityJointInterface</hardwareInterface>
+        </joint>
+        <actuator name="arm_rotate_motor">
+            <hardwareInterface>hardware_interface/VelocityJointInterface</hardwareInterface>
+            <mechanicalReduction>1</mechanicalReduction>
+        </actuator>
+    </transmission>
+    <transmission name="arm_xy_trans">
+        <type>transmission_interface/SimpleTransmission</type>
+        <joint name="arm_inner_to_outer_xy">
+            <hardwareInterface>hardware_interface/VelocityJointInterface</hardwareInterface>
+        </joint>
+        <actuator name="arm_xy_motor">
+            <hardwareInterface>hardware_interface/VelocityJointInterface</hardwareInterface>
+            <mechanicalReduction>1</mechanicalReduction>
+        </actuator>
+    </transmission>
+    <transmission name="arm_g_rotz_trans">
+        <type>transmission_interface/SimpleTransmission</type>
+        <joint name="arm_gripper_rot_z">
+            <hardwareInterface>hardware_interface/VelocityJointInterface</hardwareInterface>
+        </joint>
+        <actuator name="arm_grip_rot_z_motor">
+            <hardwareInterface>hardware_interface/VelocityJointInterface</hardwareInterface>
+            <mechanicalReduction>1</mechanicalReduction>
+        </actuator>
+    </transmission>
+    <transmission name="arm_g_roty_trans">
+        <type>transmission_interface/SimpleTransmission</type>
+        <joint name="arm_gripper_rot_y">
+            <hardwareInterface>hardware_interface/VelocityJointInterface</hardwareInterface>
+        </joint>
+        <actuator name="arm_grip_rot_y_motor">
+            <hardwareInterface>hardware_interface/VelocityJointInterface</hardwareInterface>
+            <mechanicalReduction>1</mechanicalReduction>
+        </actuator>
+    </transmission>
+    <transmission name="grip_finger_front_left_trans">
+        <type>transmission_interface/SimpleTransmission</type>
+        <joint name="gripper_base_to_finger_front_left">
+            <hardwareInterface>hardware_interface/VelocityJointInterface</hardwareInterface>
+        </joint>
+        <actuator name="gripper_base_to_finger_front_left_motor">
+            <hardwareInterface>hardware_interface/VelocityJointInterface</hardwareInterface>
+            <mechanicalReduction>1</mechanicalReduction>
+        </actuator>
+    </transmission>
+    <transmission name="grip_finger_front_right_trans">
+        <type>transmission_interface/SimpleTransmission</type>
+        <joint name="gripper_base_to_finger_front_right">
+            <hardwareInterface>hardware_interface/VelocityJointInterface</hardwareInterface>
+        </joint>
+        <actuator name="gripper_base_to_finger_front_right_motor">
+            <hardwareInterface>hardware_interface/VelocityJointInterface</hardwareInterface>
+            <mechanicalReduction>1</mechanicalReduction>
+        </actuator>
+    </transmission>
+    <transmission name="grip_finger_back_left_trans">
+        <type>transmission_interface/SimpleTransmission</type>
+        <joint name="gripper_base_to_finger_back_left">
+            <hardwareInterface>hardware_interface/VelocityJointInterface</hardwareInterface>
+        </joint>
+        <actuator name="gripper_base_to_finger_back_left_motor">
+            <hardwareInterface>hardware_interface/VelocityJointInterface</hardwareInterface>
+            <mechanicalReduction>1</mechanicalReduction>
+        </actuator>
+    </transmission>
+    <transmission name="grip_finger_back_right_trans">
+        <type>transmission_interface/SimpleTransmission</type>
+        <joint name="gripper_base_to_finger_back_right">
+            <hardwareInterface>hardware_interface/VelocityJointInterface</hardwareInterface>
+        </joint>
+        <actuator name="gripper_base_to_finger_back_right_motor">
+            <hardwareInterface>hardware_interface/VelocityJointInterface</hardwareInterface>
+            <mechanicalReduction>1</mechanicalReduction>
+        </actuator>
+    </transmission>
 </robot>

File: rosws/src/rover_description/urdf/rover.xacro.urdf (robot description, URDF)
Before this commit: robot rover, 1 links, 0 joints
Links:
- link base_link: geometry collision box size=1 0.55 0.25; visual box size=1 0.55 0.25

File: rosws/src/rover_description/urdf/wheel.xacro (robot description, xacro)
@@ -50,8 +50,25 @@
             <child link="wheel_${suffix}" />
             <axis xyz="0 1 0" />
+            <dynamics damping="0.015" friction="0.02" />
         </joint>
         <gazebo reference="wheel_leg_${suffix}">
             <material>Gazebo/Red</material>
         </gazebo>
+        <gazebo reference="wheel_${suffix}">
+            <kp value="100000" />
+            <kd value="1.0" />
+            <mu1 value="0.5" />
+            <mu2 value="0.5" />
+        </gazebo>
+        <transmission name="wheel_transmission_${suffix}">
+            <type>transmission_interface/SimpleTransmission</type>
+            <joint name="leg_to_wheel_${suffix}">
+                <hardwareInterface>hardware_interface/VelocityJointInterface</hardwareInterface>
+            </joint>
+            <actuator name="drive_motor_${suffix}">
+                <hardwareInterface>hardware_interface/VelocityJointInterface</hardwareInterface>
+                <mechanicalReduction>1</mechanicalReduction>
+            </actuator>
+        </transmission>
     </xacro:macro>
 </robot>
