Commit message: sort of works? might need to tune pids more though

File: rosws/src/rover_description/urdf/arm.xacro (robot description, xacro)
@@ -153,5 +153,5 @@
         <origin xyz="-0.05 0 0.65" rpy="0 0 0"/>
         <axis xyz="0 0 1"/>
-        <limit effort="15" velocity="0.02" lower="-0.6" upper="0.6"/>
+        <limit effort="1105" velocity="0.5" lower="-0.6" upper="0.6"/>
     </joint>
     <link name="arm_gripper_rotate_z">
@@ -204,5 +204,5 @@
         <origin xyz="0 0 -0.05" rpy="0 0 0"/>
         <axis xyz="0 1 0"/>
-        <limit effort="7" velocity="0.025" lower="-1.4" upper="1.4" />
+        <limit effort="1130" velocity="0.325" lower="-1.4" upper="1.4" />
     </joint>
     <link name="gripper_base">
@@ -284,5 +284,5 @@
         <origin xyz="0.10605 -0.10605 -0.1" rpy="0 0 -0.7853" />
         <axis xyz="0 -1 0" />
-        <limit effort="10" velocity="0.05" lower="0" upper="0.55"/>
+        <limit effort="550" velocity="0.1" lower="0" upper="0.55"/>
     </joint>
     <joint name="gripper_base_to_finger_front_right" type="revolute">
@@ -291,5 +291,5 @@
         <origin xyz="0.10605 0.10605 -0.1" rpy="0 0 0.7853" />
         <axis xyz="0 -1 0" />
-        <limit effort="10" velocity="0.05" lower="0" upper="0.55"/>
+        <limit effort="550" velocity="0.1" lower="0" upper="0.55"/>
     </joint>
     <joint name="gripper_base_to_finger_back_left" type="revolute">
@@ -298,5 +298,5 @@
         <origin xyz="-0.10605 -0.10605 -0.1" rpy="0 0 -2.35619449" />
         <axis xyz="0 -1 0" />
-        <limit effort="10" velocity="0.05" lower="0" upper="0.55"/>
+        <limit effort="550" velocity="0.1" lower="0" upper="0.55"/>
     </joint>
     <joint name="gripper_base_to_finger_back_right" type="revolute">
@@ -305,13 +305,13 @@
         <origin xyz="-0.10605 0.10605 -0.1" rpy="0 0 2.35619449" />
         <axis xyz="0 -1 0" />
-        <limit effort="10" velocity="0.05" lower="0" upper="0.55"/>
+        <limit effort="550" velocity="0.1" lower="0" upper="0.55"/>
     </joint>
     <transmission name="arm_post_rotate_trans">
         <type>transmission_interface/SimpleTransmission</type>
         <joint name="arm_base_to_post">
-            <hardwareInterface>hardware_interface/VelocityJointInterface</hardwareInterface>
+            <hardwareInterface>hardware_interface/EffortJointInterface</hardwareInterface>
         </joint>
         <actuator name="arm_rotate_motor">
-            <hardwareInterface>hardware_interface/VelocityJointInterface</hardwareInterface>
+            <hardwareInterface>hardware_interface/EffortJointInterface</hardwareInterface>
             <mechanicalReduction>1</mechanicalReduction>
         </actuator>
@@ -320,8 +320,18 @@
         <type>transmission_interface/SimpleTransmission</type>
         <joint name="arm_inner_to_outer_xy">
-            <hardwareInterface>hardware_interface/VelocityJointInterface</hardwareInterface>
+            <hardwareInterface>hardware_interface/EffortJointInterface</hardwareInterface>
         </joint>
         <actuator name="arm_xy_motor">
-            <hardwareInterface>hardware_interface/VelocityJointInterface</hardwareInterface>
+            <hardwareInterface>hardware_interface/EffortJointInterface</hardwareInterface>
+            <mechanicalReduction>1</mechanicalReduction>
+        </actuator>
+    </transmission>
+    <transmission name="arm_slide_trans">
+        <type>transmission_inteface/SimpleTransmission</type>
+        <joint name="arm_z_slide">
+            <hardwareInterface>hardware_interface/EffortJointInterface</hardwareInterface>
+        </joint>
+        <actuator name="arm_slide_motor">
+            <hardwareInterface>hardware_interface/EffortJointInterface</hardwareInterface>
             <mechanicalReduction>1</mechanicalReduction>
         </actuator>
@@ -330,8 +340,8 @@
         <type>transmission_interface/SimpleTransmission</type>
         <joint name="arm_gripper_rot_z">
-            <hardwareInterface>hardware_interface/VelocityJointInterface</hardwareInterface>
+            <hardwareInterface>hardware_interface/EffortJointInterface</hardwareInterface>
         </joint>
         <actuator name="arm_grip_rot_z_motor">
-            <hardwareInterface>hardware_interface/VelocityJointInterface</hardwareInterface>
+            <hardwareInterface>hardware_interface/EffortJointInterface</hardwareInterface>
             <mechanicalReduction>1</mechanicalReduction>
         </actuator>
@@ -340,8 +350,8 @@
         <type>transmission_interface/SimpleTransmission</type>
         <joint name="arm_gripper_rot_y">
-            <hardwareInterface>hardware_interface/VelocityJointInterface</hardwareInterface>
+            <hardwareInterface>hardware_interface/EffortJointInterface</hardwareInterface>
         </joint>
         <actuator name="arm_grip_rot_y_motor">
-            <hardwareInterface>hardware_interface/VelocityJointInterface</hardwareInterface>
+            <hardwareInterface>hardware_interface/EffortJointInterface</hardwareInterface>
             <mechanicalReduction>1</mechanicalReduction>
         </actuator>
@@ -350,8 +360,8 @@
         <type>transmission_interface/SimpleTransmission</type>
         <joint name="gripper_base_to_finger_front_left">
-            <hardwareInterface>hardware_interface/VelocityJointInterface</hardwareInterface>
+            <hardwareInterface>hardware_interface/EffortJointInterface</hardwareInterface>
         </joint>
         <actuator name="gripper_base_to_finger_front_left_motor">
-            <hardwareInterface>hardware_interface/VelocityJointInterface</hardwareInterface>
+            <hardwareInterface>hardware_interface/EffortJointInterface</hardwareInterface>
             <mechanicalReduction>1</mechanicalReduction>
         </actuator>
@@ -360,8 +370,8 @@
         <type>transmission_interface/SimpleTransmission</type>
         <joint name="gripper_base_to_finger_front_right">
-            <hardwareInterface>hardware_interface/VelocityJointInterface</hardwareInterface>
+            <hardwareInterface>hardware_interface/EffortJointInterface</hardwareInterface>
         </joint>
         <actuator name="gripper_base_to_finger_front_right_motor">
-            <hardwareInterface>hardware_interface/VelocityJointInterface</hardwareInterface>
+            <hardwareInterface>hardware_interface/EffortJointInterface</hardwareInterface>
             <mechanicalReduction>1</mechanicalReduction>
         </actuator>
@@ -370,8 +380,8 @@
         <type>transmission_interface/SimpleTransmission</type>
         <joint name="gripper_base_to_finger_back_left">
-            <hardwareInterface>hardware_interface/VelocityJointInterface</hardwareInterface>
+            <hardwareInterface>hardware_interface/EffortJointInterface</hardwareInterface>
         </joint>
         <actuator name="gripper_base_to_finger_back_left_motor">
-            <hardwareInterface>hardware_interface/VelocityJointInterface</hardwareInterface>
+            <hardwareInterface>hardware_interface/EffortJointInterface</hardwareInterface>
             <mechanicalReduction>1</mechanicalReduction>
         </actuator>
@@ -380,8 +390,8 @@
         <type>transmission_interface/SimpleTransmission</type>
         <joint name="gripper_base_to_finger_back_right">
-            <hardwareInterface>hardware_interface/VelocityJointInterface</hardwareInterface>
+            <hardwareInterface>hardware_interface/EffortJointInterface</hardwareInterface>
         </joint>
         <actuator name="gripper_base_to_finger_back_right_motor">
-            <hardwareInterface>hardware_interface/VelocityJointInterface</hardwareInterface>
+            <hardwareInterface>hardware_interface/EffortJointInterface</hardwareInterface>
             <mechanicalReduction>1</mechanicalReduction>
         </actuator>

Commit message: add documentation, might of also added the zed (might)

File: rosws/src/rover_description/urdf/arm.xacro (robot description, xacro)
@@ -153,5 +153,5 @@
         <origin xyz="-0.05 0 0.65" rpy="0 0 0"/>
         <axis xyz="0 0 1"/>
-        <limit effort="1105" velocity="0.5" lower="-0.6" upper="0.6"/>
+        <limit effort="1000" velocity="0.2" lower="-0.6" upper="0.6"/>
     </joint>
     <link name="arm_gripper_rotate_z">
@@ -204,5 +204,5 @@
         <origin xyz="0 0 -0.05" rpy="0 0 0"/>
         <axis xyz="0 1 0"/>
-        <limit effort="1130" velocity="0.325" lower="-1.4" upper="1.4" />
+        <limit effort="1000" velocity="0.4" lower="-1.4" upper="1.4" />
     </joint>
     <link name="gripper_base">
@@ -284,5 +284,5 @@
         <origin xyz="0.10605 -0.10605 -0.1" rpy="0 0 -0.7853" />
         <axis xyz="0 -1 0" />
-        <limit effort="550" velocity="0.1" lower="0" upper="0.55"/>
+        <limit effort="1000" velocity="0.4" lower="0" upper="0.55"/>
     </joint>
     <joint name="gripper_base_to_finger_front_right" type="revolute">
@@ -291,5 +291,5 @@
         <origin xyz="0.10605 0.10605 -0.1" rpy="0 0 0.7853" />
         <axis xyz="0 -1 0" />
-        <limit effort="550" velocity="0.1" lower="0" upper="0.55"/>
+        <limit effort="1000" velocity="0.4" lower="0" upper="0.55"/>
     </joint>
     <joint name="gripper_base_to_finger_back_left" type="revolute">
@@ -298,5 +298,5 @@
         <origin xyz="-0.10605 -0.10605 -0.1" rpy="0 0 -2.35619449" />
         <axis xyz="0 -1 0" />
-        <limit effort="550" velocity="0.1" lower="0" upper="0.55"/>
+        <limit effort="1000" velocity="0.4" lower="0" upper="0.55"/>
     </joint>
     <joint name="gripper_base_to_finger_back_right" type="revolute">
@@ -305,5 +305,5 @@
         <origin xyz="-0.10605 0.10605 -0.1" rpy="0 0 2.35619449" />
         <axis xyz="0 -1 0" />
-        <limit effort="550" velocity="0.1" lower="0" upper="0.55"/>
+        <limit effort="1000" velocity="0.4" lower="0" upper="0.55"/>
     </joint>
     <transmission name="arm_post_rotate_trans">
@@ -334,5 +334,5 @@
         <actuator name="arm_slide_motor">
             <hardwareInterface>hardware_interface/EffortJointInterface</hardwareInterface>
-            <mechanicalReduction>1</mechanicalReduction>
+            <mechanicalReduction>5</mechanicalReduction>
         </actuator>
     </transmission>

Commit message: demo

File: rosws/src/rover_description/urdf/arm.xacro (robot description, xacro)
@@ -23,5 +23,5 @@
         <parent link="base_link"/>
         <child link="arm_base"/>
-        <origin xyz="-0.375 0 0.25" rpy="0 0 0"/>
+        <origin xyz="0.2 0 0.25" rpy="0 0 3.14159265"/>
     </joint>
     <xacro:linkColor link="arm_base" mat="Gazebo/Red"/>
