Commit message: new ARM!!!!!

File: rosws/src/rover_description/urdf/arm.xacro (robot description, xacro)
@@ -77,5 +77,80 @@
         <axis xyz="0 0 1" />
         <origin xyz="0 0 0" rpy="0 0 0" />
-        <limit effort="2000" velocity="0.05" lower="0" upper="0.895" />
+        <limit effort="2000" velocity="1" lower="0" upper="0.895" />
+    </joint>
+    <link name="arm_xy_pole">
+        <inertial>
+            <mass value="0.32" />
+            <inertia ixx="0.00366316666667" ixy="0" ixz="0" iyy="0.00366316666667" iyz="0" izz="2.5e-05" />
+        </inertial>
+        <collision>
+            <origin xyz="0 0 -0.185" rpy="0 0 0" />
+            <geometry>
+                <cylinder length="0.37" radius="0.0125" />
+            </geometry>
+        </collision>
+        <visual>
+            <material name="White" />
+            <origin xyz="0 0 -0.185" rpy="0 0 0" />
+            <geometry>
+                <cylinder length="0.37" radius="0.0125" />
+            </geometry>
+        </visual>
+    </link>
+    <joint name="arm_slider_unit_to_arm_xy_pole" type="revolute">
+        <origin xyz="0.379 0 0" rpy="0 0 0" />
+        <axis xyz="0 0 1" />
+        <child link="arm_xy_pole" />
+        <parent link="arm_slider_unit" />
+        <limit effort="3.7" velocity="3.875" lower="-2.09" upper="2.09" />
+    </joint>
+    <link name="arm_inner">
+        <inertial>
+            <mass value="0.46" />
+            <inertia ixx="0.000155058333333" ixy="0" ixz="0" iyy="0.00252846666667" iyz="0" izz="0.00257281833333" />
+        </inertial>
+        <collision>
+            <origin xyz="0.103 0 -0.019" rpy="0 0 0" />
+            <geometry>
+                <box size="0.254 0.051 0.038" />
+            </geometry>
+        </collision>
+        <visual>
+            <material name="Blue" />
+            <origin xyz="0.103 0 -0.019" rpy="0 0 0" />
+            <geometry>
+                <box size="0.254 0.051 0.038" />
+            </geometry>
+        </visual>
+    </link>
+    <joint name="arm_xy_pole_to_arm_inner" type="fixed">
+        <child link="arm_inner" />
+        <parent link="arm_xy_pole" />
+        <origin xyz="0 0 -0.37" />
+    </joint>
+    <link name="arm_outer">
+        <inertial>
+            <mass value="0.12" />
+            <inertia ixx="1.29032e-05" ixy="0" ixz="0" iyy="0.0005127016" iyz="0" izz="0.0005127016" />
+        </inertial>
+        <collision>
+            <origin xyz="0.1125 0 -0.0127" rpy="0 0 0" />
+            <geometry>
+                <box size="0.225 0.0254 0.0254" />
+            </geometry>
+        </collision>
+        <visual>
+            <material name="Blue" />
+            <origin xyz="0.1125 0 -0.0127" rpy="0 0 0" />
+            <geometry>
+                <box size="0.225 0.0254 0.0254" />
+            </geometry>
+        </visual>
+    </link>
+    <joint name="arm_inner_to_arm_outer" type="continuous">
+        <parent link="arm_inner" />
+        <child link="arm_outer" />
+        <origin xyz="0.217 0 -0.038" rpy="0 0 0" />
+        <axis xyz="0 0 1" />
     </joint>
     <link name="gripper_base">
@@ -98,8 +173,33 @@
         </collision>
     </link>
+    <joint name="arm_outer_to_gripper_spin" type="continuous">
+        <parent link="arm_outer" />
+        <child link="gripper_spin" />
+        <origin xyz="0.220 0 -0.0254"/>
+        <axis xyz="0 0 1" />
+    </joint>
+    <link name="gripper_spin">
+        <inertial>
+            <mass value="0.08" />
+            <inertia ixx="6.16666666667e-06" ixy="0" ixz="0" iyy="6.16666666667e-06" iyz="0" izz="4e-06" />
+        </inertial>
+        <visual>
+            <material name="Red" />
+            <origin xyz="0 0 -0.00125" rpy="0 0 0" />
+            <geometry>
+                <cylinder radius="0.01" length="0.025" />
+            </geometry>
+        </visual>
+        <geometry>
+            <origin xyz="0 0 -0.00125" rpy="0 0 0" />
+            <geometry>
+                <cylinder radius="0.01" length="0.025" />
+            </geometry>
+        </geometry>
+    </link>
     <joint name="arm_to_gripper" type="fixed">
-        <parent link="arm_z_pole_front"/>
+        <parent link="gripper_spin"/>
         <child link="gripper_base"/>
-        <origin xyz="0 0 -0.05"/>
+        <origin xyz="0 0 -0.00125" rpy="0 0 0" />
     </joint>
     <xacro:macro name="finger" params="suffix">
@@ -180,17 +280,7 @@
         <limit effort="1000" velocity="0.4" lower="0" upper="0.55"/>
     </joint>
-    <transmission name="arm_post_rotate_trans">
-        <type>transmission_interface/SimpleTransmission</type>
-        <joint name="arm_base_to_post">
-            <hardwareInterface>hardware_interface/EffortJointInterface</hardwareInterface>
-        </joint>
-        <actuator name="arm_rotate_motor">
-            <hardwareInterface>hardware_interface/EffortJointInterface</hardwareInterface>
-            <mechanicalReduction>1</mechanicalReduction>
-        </actuator>
-    </transmission>
     <transmission name="arm_xy_trans">
         <type>transmission_interface/SimpleTransmission</type>
-        <joint name="arm_inner_to_outer_xy">
+        <joint name="arm_inner_to_arm_outer">
             <hardwareInterface>hardware_interface/EffortJointInterface</hardwareInterface>
         </joint>
@@ -202,5 +292,5 @@
     <transmission name="arm_slide_trans">
         <type>transmission_inteface/SimpleTransmission</type>
-        <joint name="arm_z_slide">
+        <joint name="arm_slide_pole_to_arm_slider_unit">
             <hardwareInterface>hardware_interface/EffortJointInterface</hardwareInterface>
         </joint>
@@ -210,7 +300,7 @@
         </actuator>
     </transmission>
-    <transmission name="arm_g_rotz_trans">
-        <type>transmission_interface/SimpleTransmission</type>
-        <joint name="arm_gripper_rot_z">
+    <transmission name="arm_inner_rot_trans">
+        <type>transmission_interface/SimpleTransmission</type>
+        <joint name="arm_slider_unit_to_arm_xy_pole">
             <hardwareInterface>hardware_interface/EffortJointInterface</hardwareInterface>
         </joint>
@@ -220,10 +310,10 @@
         </actuator>
     </transmission>
-    <transmission name="arm_g_roty_trans">
-        <type>transmission_interface/SimpleTransmission</type>
-        <joint name="arm_gripper_rot_y">
-            <hardwareInterface>hardware_interface/EffortJointInterface</hardwareInterface>
-        </joint>
-        <actuator name="arm_grip_rot_y_motor">
+    <transmission name="arm_spin_trans">
+        <type>transmission_interface/SimpleTransmission</type>
+        <joint name="arm_outer_to_gripper_spin">
+            <hardwareInterface>hardware_interface/EffortJointInterface</hardwareInterface>
+        </joint>
+        <actuator name="arm_grip_spin_motor">
             <hardwareInterface>hardware_interface/EffortJointInterface</hardwareInterface>
             <mechanicalReduction>1</mechanicalReduction>

Commit message: more arm

File: rosws/src/rover_description/urdf/arm.xacro (robot description, xacro)
@@ -173,111 +173,4 @@
         </collision>
     </link>
-    <joint name="arm_outer_to_gripper_spin" type="continuous">
-        <parent link="arm_outer" />
-        <child link="gripper_spin" />
-        <origin xyz="0.220 0 -0.0254"/>
-        <axis xyz="0 0 1" />
-    </joint>
-    <link name="gripper_spin">
-        <inertial>
-            <mass value="0.08" />
-            <inertia ixx="6.16666666667e-06" ixy="0" ixz="0" iyy="6.16666666667e-06" iyz="0" izz="4e-06" />
-        </inertial>
-        <visual>
-            <material name="Red" />
-            <origin xyz="0 0 -0.00125" rpy="0 0 0" />
-            <geometry>
-                <cylinder radius="0.01" length="0.025" />
-            </geometry>
-        </visual>
-        <geometry>
-            <origin xyz="0 0 -0.00125" rpy="0 0 0" />
-            <geometry>
-                <cylinder radius="0.01" length="0.025" />
-            </geometry>
-        </geometry>
-    </link>
-    <joint name="arm_to_gripper" type="fixed">
-        <parent link="gripper_spin"/>
-        <child link="gripper_base"/>
-        <origin xyz="0 0 -0.00125" rpy="0 0 0" />
-    </joint>
-    <xacro:macro name="finger" params="suffix">
-        <link name="gripper_finger_lower_${suffix}">
-            <inertial>
-                <mass value="0.08"/>
-                <inertia ixx="0.000158" ixy="0" ixz="0" iyy="0.000158" iyz="0" izz="1.6e-05"/>
-            </inertial>
-            <visual>
-                <origin xyz="0 0 -0.05" rpy="0 0 0"/>
-                <material name="White"/>
-                <geometry>
-                    <cylinder radius="0.02" length="0.1"/>
-                </geometry>
-            </visual>
-            <collision>
-                <origin xyz="0 0 -0.075" rpy="0 0 0"/>
-                <geometry>
-                    <cylinder radius="0.02" length="0.1"/>
-                </geometry>
-            </collision>
-        </link>
-        <link name="gripper_finger_upper_${suffix}">
-            <inertial>
-                <mass value="0.08"/>
-                <inertia ixx="0.000158" ixy="0" ixz="0" iyy="0.000158" iyz="0" izz="1.6e-05"/>
-            </inertial>
-            <visual>
-                <origin xyz="0 0 -0.05" rpy="0 0 0"/>
-                <material name="White"/>
-                <geometry>
-                    <cylinder radius="0.02" length="0.1"/>
-                </geometry>
-            </visual>
-            <collision>
-                <origin xyz="0 0 -0.075" rpy="0 0 0"/>
-                <geometry>
-                    <cylinder radius="0.02" length="0.1"/>
-                </geometry>
-            </collision>
-        </link>
-        <joint name="gripper_finger_link_${suffix}" type="fixed">
-            <parent link="gripper_finger_lower_${suffix}"/>
-            <child link="gripper_finger_upper_${suffix}"/>
-            <origin xyz="0 0 -0.1" rpy="0 0.55 0"/>
-        </joint>
-    </xacro:macro>
-    <xacro:finger suffix="front_left"/>
-    <xacro:finger suffix="front_right"/>
-    <xacro:finger suffix="back_left"/>
-    <xacro:finger suffix="back_right"/>
-    <joint name="gripper_base_to_finger_front_left" type="revolute">
-        <parent link="gripper_base"/>
-        <child link="gripper_finger_lower_front_left"/>
-        <origin xyz="0.10605 -0.10605 -0.1" rpy="0 0 -0.7853"/>
-        <axis xyz="0 -1 0"/>
-        <limit effort="1000" velocity="0.4" lower="0" upper="0.55"/>
-    </joint>
-    <joint name="gripper_base_to_finger_front_right" type="revolute">
-        <parent link="gripper_base"/>
-        <child link="gripper_finger_lower_front_right"/>
-        <origin xyz="0.10605 0.10605 -0.1" rpy="0 0 0.7853"/>
-        <axis xyz="0 -1 0"/>
-        <limit effort="1000" velocity="0.4" lower="0" upper="0.55"/>
-    </joint>
-    <joint name="gripper_base_to_finger_back_left" type="revolute">
-        <parent link="gripper_base"/>
-        <child link="gripper_finger_lower_back_left"/>
-        <origin xyz="-0.10605 -0.10605 -0.1" rpy="0 0 -2.35619449"/>
-        <axis xyz="0 -1 0"/>
-        <limit effort="1000" velocity="0.4" lower="0" upper="0.55"/>
-    </joint>
-    <joint name="gripper_base_to_finger_back_right" type="revolute">
-        <parent link="gripper_base"/>
-        <child link="gripper_finger_lower_back_right"/>
-        <origin xyz="-0.10605 0.10605 -0.1" rpy="0 0 2.35619449"/>
-        <axis xyz="0 -1 0"/>
-        <limit effort="1000" velocity="0.4" lower="0" upper="0.55"/>
-    </joint>
     <transmission name="arm_outer_xy_trans">
         <type>transmission_interface/SimpleTransmission</type>
@@ -310,53 +203,3 @@
         </actuator>
     </transmission>
-    <transmission name="arm_spin_trans">
-        <type>transmission_interface/SimpleTransmission</type>
-        <joint name="arm_outer_to_gripper_spin">
-            <hardwareInterface>hardware_interface/EffortJointInterface</hardwareInterface>
-        </joint>
-        <actuator name="arm_grip_spin_motor">
-            <hardwareInterface>hardware_interface/EffortJointInterface</hardwareInterface>
-            <mechanicalReduction>1</mechanicalReduction>
-        </actuator>
-    </transmission>
-    <transmission name="grip_finger_front_left_trans">
-        <type>transmission_interface/SimpleTransmission</type>
-        <joint name="gripper_base_to_finger_front_left">
-            <hardwareInterface>hardware_interface/EffortJointInterface</hardwareInterface>
-        </joint>
-        <actuator name="gripper_base_to_finger_front_left_motor">
-            <hardwareInterface>hardware_interface/EffortJointInterface</hardwareInterface>
-            <mechanicalReduction>1</mechanicalReduction>
-        </actuator>
-    </transmission>
-    <transmission name="grip_finger_front_right_trans">
-        <type>transmission_interface/SimpleTransmission</type>
-        <joint name="gripper_base_to_finger_front_right">
-            <hardwareInterface>hardware_interface/EffortJointInterface</hardwareInterface>
-        </joint>
-        <actuator name="gripper_base_to_finger_front_right_motor">
-            <hardwareInterface>hardware_interface/EffortJointInterface</hardwareInterface>
-            <mechanicalReduction>1</mechanicalReduction>
-        </actuator>
-    </transmission>
-    <transmission name="grip_finger_back_left_trans">
-        <type>transmission_interface/SimpleTransmission</type>
-        <joint name="gripper_base_to_finger_back_left">
-            <hardwareInterface>hardware_interface/EffortJointInterface</hardwareInterface>
-        </joint>
-        <actuator name="gripper_base_to_finger_back_left_motor">
-            <hardwareInterface>hardware_interface/EffortJointInterface</hardwareInterface>
-            <mechanicalReduction>1</mechanicalReduction>
-        </actuator>
-    </transmission>
-    <transmission name="grip_finger_back_right_trans">
-        <type>transmission_interface/SimpleTransmission</type>
-        <joint name="gripper_base_to_finger_back_right">
-            <hardwareInterface>hardware_interface/EffortJointInterface</hardwareInterface>
-        </joint>
-        <actuator name="gripper_base_to_finger_back_right_motor">
-            <hardwareInterface>hardware_interface/EffortJointInterface</hardwareInterface>
-            <mechanicalReduction>1</mechanicalReduction>
-        </actuator>
-    </transmission>
 </robot>

Commit message: current version

File: rosws/src/rover_description/urdf/arm.xacro (robot description, xacro)
@@ -148,4 +148,29 @@
         </visual>
     </link>
+    <link name="grip_spin">
+        <inertial>
+            <mass value="0.05" />
+            <inertia ixx="1.29032e-05" ixy="0" ixz="0" iyy="0.0005127016" iyz="0" izz="0.0005127016" />
+        </inertial>
+        <collision>
+            <origin xyz="0 0 -0.05" rpy="0 0 0" />
+            <geometry>
+                <cylinder radius="0.025" length="0.1" />
+            </geometry>
+        </collision>
+        <visual>
+            <material name="Blue" />
+            <origin xyz="0 0 -0.05" rpy="0 0 0" />
+            <geometry>
+                <cylinder radius="0.025" length="0.1" />
+            </geometry>
+        </visual>
+    </link>
+    <joint name="arm_outer_to_grip_spin" type="continuous">
+        <parent link="arm_outer" />
+        <child link="grip_spin" />
+        <origin xyz="0.225 0 -0.0127" rpy="0 0 0" />
+        <axis xyz="0 0 1" />
+    </joint>
     <joint name="arm_inner_to_arm_outer" type="continuous">
         <parent link="arm_inner" />
@@ -154,23 +179,4 @@
         <axis xyz="0 0 1" />
     </joint>
-    <link name="gripper_base">
-        <inertial>
-            <mass value="0.3"/>
-            <inertia ixx="0.0019375" ixy="0" ixz="0" iyy="0.0019375" iyz="0" izz="0.003375"/>
-        </inertial>
-        <visual>
-            <material name="Yellow"/>
-            <origin xyz="0 0 -0.05" rpy="0 0 0"/>
-            <geometry>
-                <cylinder length="0.1" radius="0.15"/>
-            </geometry>
-        </visual>
-        <collision>
-            <origin xyz="0 0 -0.05" rpy="0 0 0"/>
-            <geometry>
-                <cylinder length="0.1" radius="0.15"/>
-            </geometry>
-        </collision>
-    </link>
     <transmission name="arm_outer_xy_trans">
         <type>transmission_interface/SimpleTransmission</type>
@@ -203,3 +209,13 @@
         </actuator>
     </transmission>
+    <transmission name="arm_sping">
+        <type>transmission_interface/SimpleTransmission</type>
+        <joint name="arm_outer_to_grip_spin">
+            <hardwareInterface>hardware_interface/EffortJointInterface</hardwareInterface>
+        </joint>
+        <actuator name="arm_spin_inner_motor">
+            <hardwareInterface>hardware_interface/EffortJointInterface</hardwareInterface>
+            <mechanicalReduction>1</mechanicalReduction>
+        </actuator>
+    </transmission>
 </robot>
