Commit message: reformat arm to a better format

File: rosws/src/rover_description/urdf/arm.xacro (robot description, xacro)
@@ -5,5 +5,5 @@
             <inertial>
                 <mass value="0.22"/>
-                <inertia ixx="0.0183532929708" ixy="0" ixz="0" iyy="0.0183532929708" iyz="0" izz="3.9919275e-05" />
+                <inertia ixx="0.0183532929708" ixy="0" ixz="0" iyy="0.0183532929708" iyz="0" izz="3.9919275e-05"/>
             </inertial>
             <visual>
@@ -22,171 +22,111 @@
         </link>
         <joint name="base_link_to_arm_z_pole_${suffix}" type="fixed">
-            <parent link="base_link" />
-            <child link="arm_z_pole_${suffix}" />
-            <origin xyz="${x} 0 0.25" />
+            <parent link="base_link"/>
+            <child link="arm_z_pole_${suffix}"/>
+            <origin xyz="${x} 0 0.25"/>
         </joint>
     </xacro:macro>
-    <xacro:arm_z_pole x="0.3" suffix="back" />
-    <xacro:arm_z_pole x="0.45" suffix="front" />
+    <xacro:arm_z_pole x="0.3" suffix="back"/>
+    <xacro:arm_z_pole x="0.45" suffix="front"/>
     <link name="arm_z_pole_endcap">
         <inertial>
-            <mass value="0.39" />
-            <inertia ixx="0.0001105" ixy="0" ixz="0" iyy="0.00132925" iyz="0" izz="0.00138125" />
+            <mass value="0.39"/>
+            <inertia ixx="0.0001105" ixy="0" ixz="0" iyy="0.00132925" iyz="0" izz="0.00138125"/>
         </inertial>
         <visual>
-            <origin xyz="0.075 0 0.03" rpy="0 0 0" />
-            <material name="Yellow" />
+            <origin xyz="0.075 0 0.03" rpy="0 0 0"/>
+            <material name="Yellow"/>
             <geometry>
-                <box size="0.2 0.05 0.03" />
+                <box size="0.2 0.05 0.03"/>
             </geometry>
         </visual>
         <collision>
-            <origin xyz="0.075 0 0.03" rpy="0 0 0" />
+            <origin xyz="0.075 0 0.03" rpy="0 0 0"/>
             <geometry>
-                <box size="0.2 0.05 0.03" />
+                <box size="0.2 0.05 0.03"/>
             </geometry>
         </collision>
     </link>
     <joint name="arm_z_pole_to_arm_z_pole_endcap" type="fixed">
-        <parent link="arm_z_pole_back" />
-        <child link="arm_z_pole_endcap" />
-        <origin xyz="0 0 0.97" />
+        <parent link="arm_z_pole_back"/>
+        <child link="arm_z_pole_endcap"/>
+        <origin xyz="0 0 0.97"/>
     </joint>
     <link name="arm_slider_unit">
         <inertial>
-            <mass value="1.26" />
-            <inertia ixx="0.002625" ixy="0" ixz="0" iyy="0.021777" iyz="0" izz="0.019677" />
+            <mass value="1.26"/>
+            <inertia ixx="0.002625" ixy="0" ixz="0" iyy="0.021777" iyz="0" izz="0.019677"/>
         </inertial>
         <visual>
-            <material name="Green" />
-            <origin xyz="0.19 0 0.075" rpy="0 0 0" />
+            <material name="Green"/>
+            <origin xyz="0.19 0 0.075" rpy="0 0 0"/>
             <geometry>
-                <box size="0.43 0.05 0.15" />
+                <box size="0.43 0.05 0.15"/>
             </geometry>
         </visual>
         <collision>
-            <origin xyz="0.19 0 0.075" rpy="0 0 0" />
+            <origin xyz="0.19 0 0.075" rpy="0 0 0"/>
             <geometry>
-                <box size="0.43 0.05 0.15" />
+                <box size="0.43 0.05 0.15"/>
             </geometry>
         </collision>
     </link>
     <joint name="arm_slide_pole_to_arm_slider_unit" type="prismatic">
-        <parent link="arm_z_pole_back" />
-        <child link="arm_slider_unit" />
-        <axis xyz="0 0 1" />
-        <origin xyz="0 0 0" rpy="0 0 0" />
-        <limit effort="2000" velocity="1" lower="0" upper="0.895" />
+        <parent link="arm_z_pole_back"/>
+        <child link="arm_slider_unit"/>
+        <axis xyz="0 0 1"/>
+        <origin xyz="0 0 0" rpy="0 0 0"/>
+        <limit effort="2000" velocity="1" lower="0" upper="0.895"/>
     </joint>
     <link name="arm_xy_pole">
         <inertial>
-            <mass value="0.32" />
-            <inertia ixx="0.00366316666667" ixy="0" ixz="0" iyy="0.00366316666667" iyz="0" izz="2.5e-05" />
+            <mass value="0.32"/>
+            <inertia ixx="0.00366316666667" ixy="0" ixz="0" iyy="0.00366316666667" iyz="0" izz="2.5e-05"/>
         </inertial>
         <collision>
-            <origin xyz="0 0 -0.185" rpy="0 0 0" />
+            <origin xyz="0 0 -0.185" rpy="0 0 0"/>
             <geometry>
-                <cylinder length="0.37" radius="0.0125" />
+                <cylinder length="0.37" radius="0.0125"/>
             </geometry>
         </collision>
         <visual>
-            <material name="White" />
-            <origin xyz="0 0 -0.185" rpy="0 0 0" />
+            <material name="White"/>
+            <origin xyz="0 0 -0.185" rpy="0 0 0"/>
             <geometry>
-                <cylinder length="0.37" radius="0.0125" />
+                <cylinder length="0.37" radius="0.0125"/>
             </geometry>
         </visual>
     </link>
     <joint name="arm_slider_unit_to_arm_xy_pole" type="revolute">
-        <origin xyz="0.379 0 0" rpy="0 0 0" />
-        <axis xyz="0 0 1" />
-        <child link="arm_xy_pole" />
-        <parent link="arm_slider_unit" />
-        <limit effort="3.7" velocity="3.875" lower="-2.09" upper="2.09" />
+        <origin xyz="0.379 0 0" rpy="0 0 0"/>
+        <axis xyz="0 0 1"/>
+        <child link="arm_xy_pole"/>
+        <parent link="arm_slider_unit"/>
+        <limit effort="3.7" velocity="3.875" lower="-2.09" upper="2.09"/>
     </joint>
     <link name="arm_inner">
         <inertial>
-            <mass value="0.46" />
-            <inertia ixx="0.000155058333333" ixy="0" ixz="0" iyy="0.00252846666667" iyz="0" izz="0.00257281833333" />
+            <mass value="0.46"/>
+            <inertia ixx="0.000155058333333" ixy="0" ixz="0" iyy="0.00252846666667" iyz="0" izz="0.00257281833333"/>
         </inertial>
         <collision>
-            <origin xyz="0.103 0 -0.019" rpy="0 0 0" />
+            <origin xyz="0.103 0 -0.019" rpy="0 0 0"/>
             <geometry>
-                <box size="0.254 0.051 0.038" />
+                <box size="0.254 0.051 0.038"/>
             </geometry>
         </collision>
         <visual>
-            <material name="Blue" />
-            <origin xyz="0.103 0 -0.019" rpy="0 0 0" />
+            <material name="Blue"/>
+            <origin xyz="0.103 0 -0.019" rpy="0 0 0"/>
             <geometry>
-                <box size="0.254 0.051 0.038" />
+                <box size="0.254 0.051 0.038"/>
             </geometry>
         </visual>
     </link>
     <joint name="arm_xy_pole_to_arm_inner" type="fixed">
-        <child link="arm_inner" />
-        <parent link="arm_xy_pole" />
-        <origin xyz="0 0 -0.37" />
+        <child link="arm_inner"/>
+        <parent link="arm_xy_pole"/>
+        <origin xyz="0 0 -0.37"/>
     </joint>
-    <link name="arm_outer">
-        <inertial>
-            <mass value="0.12" />
-            <inertia ixx="1.29032e-05" ixy="0" ixz="0" iyy="0.0005127016" iyz="0" izz="0.0005127016" />
-        </inertial>
-        <collision>
-            <origin xyz="0.1125 0 -0.0127" rpy="0 0 0" />
-            <geometry>
-                <box size="0.225 0.0254 0.0254" />
-            </geometry>
-        </collision>
-        <visual>
-            <material name="Blue" />
-            <origin xyz="0.1125 0 -0.0127" rpy="0 0 0" />
-            <geometry>
-                <box size="0.225 0.0254 0.0254" />
-            </geometry>
-        </visual>
-    </link>
-    <link name="grip_spin">
-        <inertial>
-            <mass value="0.05" />
-            <inertia ixx="1.29032e-05" ixy="0" ixz="0" iyy="0.0005127016" iyz="0" izz="0.0005127016" />
-        </inertial>
-        <collision>
-            <origin xyz="0 0 -0.05" rpy="0 0 0" />
-            <geometry>
-                <cylinder radius="0.025" length="0.1" />
-            </geometry>
-        </collision>
-        <visual>
-            <material name="Blue" />
-            <origin xyz="0 0 -0.05" rpy="0 0 0" />
-            <geometry>
-                <cylinder radius="0.025" length="0.1" />
-            </geometry>
-        </visual>
-    </link>
-    <joint name="arm_outer_to_grip_spin" type="continuous">
-        <parent link="arm_outer" />
-        <child link="grip_spin" />
-        <origin xyz="0.225 0 -0.0127" rpy="0 0 0" />
-        <axis xyz="0 0 1" />
-    </joint>
-    <joint name="arm_inner_to_arm_outer" type="continuous">
-        <parent link="arm_inner" />
-        <child link="arm_outer" />
-        <origin xyz="0.217 0 -0.038" rpy="0 0 0" />
-        <axis xyz="0 0 1" />
-    </joint>
-    <transmission name="arm_outer_xy_trans">
-        <type>transmission_interface/SimpleTransmission</type>
-        <joint name="arm_inner_to_arm_outer">
-            <hardwareInterface>hardware_interface/EffortJointInterface</hardwareInterface>
-        </joint>
-        <actuator name="arm_xy_outer_motor">
-            <hardwareInterface>hardware_interface/EffortJointInterface</hardwareInterface>
-            <mechanicalReduction>1</mechanicalReduction>
-        </actuator>
-    </transmission>
     <transmission name="arm_slide_trans">
         <type>transmission_inteface/SimpleTransmission</type>
@@ -209,13 +149,7 @@
         </actuator>
     </transmission>
-    <transmission name="arm_sping">
-        <type>transmission_interface/SimpleTransmission</type>
-        <joint name="arm_outer_to_grip_spin">
-            <hardwareInterface>hardware_interface/EffortJointInterface</hardwareInterface>
-        </joint>
-        <actuator name="arm_spin_inner_motor">
-            <hardwareInterface>hardware_interface/EffortJointInterface</hardwareInterface>
-            <mechanicalReduction>1</mechanicalReduction>
-        </actuator>
-    </transmission>
+    <xacro:property name="gripper_type" value="$(arg gripper_type)" />
+    <xacro:if value="${gripper_type != 'no_gripper'}">
+        <xacro:include filename="grippers/$(arg gripper_type).xacro"/>
+    </xacro:if>
 </robot>
