Commit message: Arm software (#14)
SQUAAAAASH it and merge it

woopeee


* Start new arm

including new stars like:

   - the poles
   - the box
   - the encap

and returning players like:

   - the gripper

* new ARM!!!!!

* better naming

* move eml_uberdriver

* almost done docs for eml_uberdriver

WARNING: this will probably get moved out to rtd for a seperate system, but for now
it is staying here

* fix uberfirmware

* START ARM

* begin work on rover arm,

* more arm

* stuff in progress

* current version

* asdf

* reformat arm to a better format

* add science gripper

* add science controllers

* reorg arm_hw

* begin science arm

* more arm

* tune pids better

* begin as

* asdf - asdf

* add various things

* change outdoor_world to support multiple grippers

a sane commit message?

* further change

* start work on new arm software

for test

it'll work
i promise
no i dont
neveer mind

* maybe working code for arm

* changed the address to match hardware

* stop spamming a you git

* modify

GABE WHY

* yayyayayayaya

why am i so tired

* add motor constants

* hmmmm

* 2 is not wired?

* HUZZAH (it works)

this is a matthew commit, under gabe's account(maybe)

* last minute changes

File: rosws/src/rover_description/urdf/arm.xacro (robot description, xacro)
@@ -1,399 +1,155 @@
 <?xml version="1.0" ?>
 <robot xmlns:xacro="http://www.ros.org/wiki/xacro">
-    <link name="arm_base">
+    <xacro:macro name="arm_z_pole" params="suffix x">
+        <link name="arm_z_pole_${suffix}">
+            <inertial>
+                <mass value="0.22"/>
+                <inertia ixx="0.0183532929708" ixy="0" ixz="0" iyy="0.0183532929708" iyz="0" izz="3.9919275e-05"/>
+            </inertial>
+            <visual>
+                <origin xyz="0 0 0.485" rpy="0 0 0"/>
+                <material name="Red"/>
+                <geometry>
+                    <cylinder length="0.97" radius="0.01905"/>
+                </geometry>
+            </visual>
+            <collision>
+                <origin xyz="0 0 0.485" rpy="0 0 0"/>
+                <geometry>
+                    <cylinder length="0.97" radius="0.01905"/>
+                </geometry>
+            </collision>
+        </link>
+        <joint name="base_link_to_arm_z_pole_${suffix}" type="fixed">
+            <parent link="base_link"/>
+            <child link="arm_z_pole_${suffix}"/>
+            <origin xyz="${x} 0 0.25"/>
+        </joint>
+    </xacro:macro>
+    <xacro:arm_z_pole x="0.3" suffix="back"/>
+    <xacro:arm_z_pole x="0.45" suffix="front"/>
+    <link name="arm_z_pole_endcap">
         <inertial>
-            <mass value="0.2"/>
-            <inertia ixx="0.000416666666667" ixy="0" ixz="0" iyy="0.000416666666667" iyz="0" izz="0.00075"/>
+            <mass value="0.39"/>
+            <inertia ixx="0.0001105" ixy="0" ixz="0" iyy="0.00132925" iyz="0" izz="0.00138125"/>
         </inertial>
         <visual>
-            <origin xyz="0 0 0.025" rpy="0 0 0"/>
-            <material name="Red"/>
+            <origin xyz="0.075 0 0.03" rpy="0 0 0"/>
+            <material name="Yellow"/>
             <geometry>
-                <box size="0.15 0.15 0.05"/>
+                <box size="0.2 0.05 0.03"/>
             </geometry>
         </visual>
         <collision>
-            <origin xyz="0 0 0.025" rpy="0 0 0"/>
+            <origin xyz="0.075 0 0.03" rpy="0 0 0"/>
             <geometry>
-                <box size="0.15 0.15 0.05"/>
+                <box size="0.2 0.05 0.03"/>
             </geometry>
         </collision>
     </link>
-    <joint name="base_to_arm_base" type="fixed">
-        <parent link="base_link"/>
-        <child link="arm_base"/>
-        <origin xyz="0.2 0 0.25" rpy="0 0 3.14159265"/>
+    <joint name="arm_z_pole_to_arm_z_pole_endcap" type="fixed">
+        <parent link="arm_z_pole_back"/>
+        <child link="arm_z_pole_endcap"/>
+        <origin xyz="0 0 0.97"/>
     </joint>
-    <xacro:linkColor link="arm_base" mat="Gazebo/Red"/>
-    <link name="arm_post">
+    <link name="arm_slider_unit">
         <inertial>
-            <mass value="1.5"/>
-            <inertia ixx="0.02135" ixy="0" ixz="0" iyy="0.02135" iyz="0" izz="0.0027"/>
+            <mass value="1.26"/>
+            <inertia ixx="0.002625" ixy="0" ixz="0" iyy="0.021777" iyz="0" izz="0.019677"/>
         </inertial>
         <visual>
-            <origin xyz="0 0 0.2" rpy="0 0 0"/>
-            <material name="Blue"/>
+            <material name="Green"/>
+            <origin xyz="0.19 0 0.075" rpy="0 0 0"/>
             <geometry>
-                <cylinder radius="0.06" length="0.4"/>
+                <box size="0.43 0.05 0.15"/>
             </geometry>
         </visual>
         <collision>
-            <origin xyz="0 0 0.2" rpy="0 0 0"/>
+            <origin xyz="0.19 0 0.075" rpy="0 0 0"/>
             <geometry>
-                <cylinder radius="0.06" length="0.4"/>
+                <box size="0.43 0.05 0.15"/>
             </geometry>
         </collision>
     </link>
-    <xacro:linkColor link="arm_post" mat="Gazebo/Blue"/>
-    <joint name="arm_base_to_post" type="continuous">
-        <parent link="arm_base"/>
-        <child link="arm_post"/>
-        <origin xyz="0 0 0.05"/>
+    <xacro:linkColor link="arm_slider_unit" mat="Gazebo/Blue" />
+    <joint name="arm_slide_pole_to_arm_slider_unit" type="prismatic">
+        <parent link="arm_z_pole_back"/>
+        <child link="arm_slider_unit"/>
         <axis xyz="0 0 1"/>
+        <origin xyz="0 0 0" rpy="0 0 0"/>
+        <limit effort="2000" velocity="1" lower="0" upper="0.895"/>
     </joint>
-    <link name="arm_inner_xy">
+    <link name="arm_xy_pole">
         <inertial>
-            <mass value="0.2"/>
-            <inertia ixx="0.00618" ixy="0" ixz="0" iyy="0.00618" iyz="0" izz="0.00036"/>
+            <mass value="0.32"/>
+            <inertia ixx="0.00366316666667" ixy="0" ixz="0" iyy="0.00366316666667" iyz="0" izz="2.5e-05"/>
         </inertial>
+        <collision>
+            <origin xyz="0 0 -0.185" rpy="0 0 0"/>
+            <geometry>
+                <cylinder length="0.37" radius="0.0125"/>
+            </geometry>
+        </collision>
         <visual>
-            <origin xyz="0 0 0.3" rpy="0 0 0"/>
-            <material name="Yellow"/>
+            <material name="White"/>
+            <origin xyz="0 0 -0.185" rpy="0 0 0"/>
             <geometry>
-                <cylinder radius="0.06" length="0.6"/>
+                <cylinder length="0.37" radius="0.0125"/>
             </geometry>
         </visual>
+    </link>
+    <joint name="arm_slider_unit_to_arm_xy_pole" type="revolute">
+        <origin xyz="0.379 0 0" rpy="0 0 0"/>
+        <axis xyz="0 0 1"/>
+        <child link="arm_xy_pole"/>
+        <parent link="arm_slider_unit"/>
+        <limit effort="3.7" velocity="3.875" lower="-2.09" upper="2.09"/>
+    </joint>
+    <link name="arm_inner">
+        <inertial>
+            <mass value="0.46"/>
+            <inertia ixx="0.000155058333333" ixy="0" ixz="0" iyy="0.00252846666667" iyz="0" izz="0.00257281833333"/>
+        </inertial>
         <collision>
-            <origin xyz="0 0 0.3" rpy="0 0 0"/>
+            <origin xyz="0.103 0 -0.019" rpy="0 0 0"/>
             <geometry>
-                <cylinder radius="0.06" length="0.6"/>
+                <box size="0.254 0.051 0.038"/>
             </geometry>
         </collision>
-    </link>
-    <joint name="arm_post_to_inner_xy" type="fixed">
-        <parent link="arm_post"/>
-        <child link="arm_inner_xy"/>
-        <origin xyz="0 0 0.4" rpy="0 -1.5708 0"/>
-    </joint>
-    <xacro:linkColor link="arm_inner_xy" mat="Gazebo/Yellow"/>
-    <link name="arm_outer_xy">
-        <inertial>
-            <mass value="0.2"/>
-            <inertia ixx="0.00618" ixy="0" ixz="0" iyy="0.00618" iyz="0" izz="0.00036"/>
-        </inertial>
         <visual>
-            <origin xyz="0 0 0.3" rpy="0 0 0"/>
-            <material name="Yellow"/>
+            <material name="Blue"/>
+            <origin xyz="0.103 0 -0.019" rpy="0 0 0"/>
             <geometry>
-                <cylinder radius="0.06" length="0.6"/>
+                <box size="0.254 0.051 0.038"/>
             </geometry>
         </visual>
-        <collision>
-            <origin xyz="0 0 0.3" rpy="0 0 0"/>
-            <geometry>
-                <cylinder radius="0.06" length="0.6"/>
-            </geometry>
-        </collision>
     </link>
-    <xacro:linkColor link="arm_outer_xy" mat="Gazebo/Yellow"/>
-    <joint name="arm_inner_to_outer_xy" type="continuous">
-        <parent link="arm_inner_xy"/>
-        <child link="arm_outer_xy"/>
-        <origin xyz="0 0 0.6" rpy="0 0 0"/>
-        <axis xyz="1 0 0"/>
+    <xacro:linkColor link="arm_inner" mat="Gazebo/Red" />
+    <joint name="arm_xy_pole_to_arm_inner" type="fixed">
+        <child link="arm_inner"/>
+        <parent link="arm_xy_pole"/>
+        <origin xyz="0 0 -0.37"/>
     </joint>
-    <link name="arm_slide_holder">
-        <inertial>
-            <mass value="0.15"/>
-            <inertia ixx="0.00025" ixy="0" ixz="0" iyy="0.00025" iyz="0" izz="0.00025"/>
-        </inertial>
-        <visual>
-            <origin xyz="-0.05 0 0" rpy="0 0 0"/>
-            <material name="Red"/>
-            <geometry>
-                <box size="0.1 0.1 0.1"/>
-            </geometry>
-        </visual>
-        <collision>
-            <origin xyz="0 0 0.05" rpy="0 0 0"/>
-            <geometry>
-                <box size="0.1 0.1 0.1"/>
-            </geometry>
-        </collision>
-    </link>
-    <xacro:linkColor mat="Gazebo/Red" link="arm_slide_holder"/>
-    <joint name="arm_outer_xy_to_slide_holder" type="fixed">
-        <parent link="arm_outer_xy"/>
-        <child link="arm_slide_holder"/>
-        <origin xyz="0 0 0.6" rpy="0 1.5708 0"/>
-    </joint>
-    <link name="arm_z">
-        <inertial>
-            <mass value="0.2"/>
-            <inertia ixx="0.0141233333333" ixy="0" ixz="0" iyy="0.0141233333333" iyz="0" izz="8e-05"/>
-        </inertial>
-        <visual>
-            <material name="Blue"/>
-            <origin xyz="0 0 -0.65" rpy="0 0 0"/>
-            <geometry>
-                <cylinder length="1.3" radius="0.04"/>
-            </geometry>
-        </visual>
-        <collision>
-            <origin xyz="0 0 -0.65" rpy="0 0 0"/>
-            <geometry>
-                <cylinder length="1.3" radius="0.04"/>
-            </geometry>
-        </collision>
-    </link>
-    <xacro:linkColor link="arm_z" mat="Gazebo/Blue"/>
-    <joint name="arm_z_slide" type="prismatic">
-        <parent link="arm_slide_holder"/>
-        <child link="arm_z"/>
-        <origin xyz="-0.05 0 0.65" rpy="0 0 0"/>
-        <axis xyz="0 0 1"/>
-        <limit effort="1000" velocity="0.2" lower="-0.6" upper="0.6"/>
-    </joint>
-    <link name="arm_gripper_rotate_z">
-        <inertial>
-            <mass value="0.1"/>
-            <inertia ixx="4.08333333333e-05" ixy="0" ixz="0" iyy="4.08333333333e-05" iyz="0" izz="8e-05"/>
-        </inertial>
-        <visual>
-            <material name="White"/>
-            <origin xyz="0 0 -0.025" rpy="0 0 0"/>
-            <geometry>
-                <cylinder radius="0.04" length="0.05"/>
-            </geometry>
-        </visual>
-        <collision>
-            <origin xyz="0 0 -0.025" rpy="0 0 0"/>
-            <geometry>
-                <cylinder radius="0.04" length="0.05"/>
-            </geometry>
-        </collision>
-    </link>
-    <joint name="arm_gripper_rot_z" type="continuous">
-        <parent link="arm_z"/>
-        <child link="arm_gripper_rotate_z"/>
-        <origin xyz="0 0 -1.3" rpy="0 0 0"/>
-        <axis xyz="0 0 1"/>
-    </joint>
-    <link name="arm_gripper_rotate_y">
-        <inertial>
-            <mass value="0.1"/>
-            <inertia ixx="4.08333333333e-05" ixy="0" ixz="0" iyy="4.08333333333e-05" iyz="0" izz="8e-05"/>
-        </inertial>
-        <visual>
-            <material name="White"/>
-            <origin xyz="0 0 -0.025" rpy="0 0 0"/>
-            <geometry>
-                <cylinder radius="0.04" length="0.05"/>
-            </geometry>
-        </visual>
-        <collision>
-            <origin xyz="0 0 -0.025" rpy="0 0 0"/>
-            <geometry>
-                <cylinder radius="0.04" length="0.05"/>
-            </geometry>
-        </collision>
-    </link>
-    <joint name="arm_gripper_rot_y" type="revolute">
-        <parent link="arm_gripper_rotate_z"/>
-        <child link="arm_gripper_rotate_y"/>
-        <origin xyz="0 0 -0.05" rpy="0 0 0"/>
-        <axis xyz="0 1 0"/>
-        <limit effort="1000" velocity="0.4" lower="-1.4" upper="1.4" />
-    </joint>
-    <link name="gripper_base">
-        <inertial>
-            <mass value="0.3" />
-            <inertia ixx="0.0019375" ixy="0" ixz="0" iyy="0.0019375" iyz="0" izz="0.003375" />
-        </inertial>
-        <visual>
-            <material name="Yellow" />
-            <origin xyz="0 0 -0.05" rpy="0 0 0" />
-            <geometry>
-                <cylinder length="0.1" radius="0.15" />
-            </geometry>
-        </visual>
-        <collision>
-            <origin xyz="0 0 -0.05" rpy="0 0 0" />
-            <geometry>
-                <cylinder length="0.1" radius="0.15" />
-            </geometry>
-        </collision>
-    </link>
-    <joint name="arm_to_gripper" type="fixed">
-        <parent link="arm_gripper_rotate_y" />
-        <child link="gripper_base" />
-        <origin xyz="0 0 -0.05" />
-    </joint>
-    <xacro:macro name="finger" params="suffix">
-        <link name="gripper_finger_lower_${suffix}">
-            <inertial>
-                <mass value="0.08" />
-                <inertia ixx="0.000158" ixy="0" ixz="0" iyy="0.000158" iyz="0" izz="1.6e-05" />
-            </inertial>
-            <visual>
-                <origin xyz="0 0 -0.05" rpy="0 0 0" />
-                <material name="White" />
-                <geometry>
-                    <cylinder radius="0.02" length="0.1" />
-                </geometry>
-            </visual>
-            <collision>
-                <origin xyz="0 0 -0.075" rpy="0 0 0" />
-                <geometry>
-                    <cylinder radius="0.02" length="0.1" />
-                </geometry>
-            </collision>
-        </link>
-        <link name="gripper_finger_upper_${suffix}">
-            <inertial>
-                <mass value="0.08" />
-                <inertia ixx="0.000158" ixy="0" ixz="0" iyy="0.000158" iyz="0" izz="1.6e-05" />
-            </inertial>
-            <visual>
-                <origin xyz="0 0 -0.05" rpy="0 0 0" />
-                <material name="White" />
-                <geometry>
-                    <cylinder radius="0.02" length="0.1" />
-                </geometry>
-            </visual>
-            <collision>
-                <origin xyz="0 0 -0.075" rpy="0 0 0" />
-                <geometry>
-                    <cylinder radius="0.02" length="0.1" />
-                </geometry>
-            </collision>
-        </link>
-        <joint name="gripper_finger_link_${suffix}" type="fixed">
-            <parent link="gripper_finger_lower_${suffix}" />
-            <child  link="gripper_finger_upper_${suffix}" />
-            <origin xyz="0 0 -0.1" rpy="0 0.55 0" />
-        </joint>
-    </xacro:macro>
-    <xacro:finger suffix="front_left" />
-    <xacro:finger suffix="front_right" />
-    <xacro:finger suffix="back_left" />
-    <xacro:finger suffix="back_right" />
-    <joint name="gripper_base_to_finger_front_left" type="revolute">
-        <parent link="gripper_base" />
-        <child link="gripper_finger_lower_front_left" />
-        <origin xyz="0.10605 -0.10605 -0.1" rpy="0 0 -0.7853" />
-        <axis xyz="0 -1 0" />
-        <limit effort="1000" velocity="0.4" lower="0" upper="0.55"/>
-    </joint>
-    <joint name="gripper_base_to_finger_front_right" type="revolute">
-        <parent link="gripper_base" />
-        <child link="gripper_finger_lower_front_right" />
-        <origin xyz="0.10605 0.10605 -0.1" rpy="0 0 0.7853" />
-        <axis xyz="0 -1 0" />
-        <limit effort="1000" velocity="0.4" lower="0" upper="0.55"/>
-    </joint>
-    <joint name="gripper_base_to_finger_back_left" type="revolute">
-        <parent link="gripper_base" />
-        <child link="gripper_finger_lower_back_left" />
-        <origin xyz="-0.10605 -0.10605 -0.1" rpy="0 0 -2.35619449" />
-        <axis xyz="0 -1 0" />
-        <limit effort="1000" velocity="0.4" lower="0" upper="0.55"/>
-    </joint>
-    <joint name="gripper_base_to_finger_back_right" type="revolute">
-        <parent link="gripper_base" />
-        <child link="gripper_finger_lower_back_right" />
-        <origin xyz="-0.10605 0.10605 -0.1" rpy="0 0 2.35619449" />
-        <axis xyz="0 -1 0" />
-        <limit effort="1000" velocity="0.4" lower="0" upper="0.55"/>
-    </joint>
-    <transmission name="arm_post_rotate_trans">
+    <transmission name="arm_slide_trans">
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
Commit message: add les units

File: rosws/src/rover_description/urdf/arm.xacro (robot description, xacro)
@@ -24,9 +24,9 @@
             <parent link="base_link"/>
             <child link="arm_z_pole_${suffix}"/>
-            <origin xyz="${x} 0 0.25"/>
+            <origin xyz="${x} 0 0.1"/>
         </joint>
     </xacro:macro>
-    <xacro:arm_z_pole x="0.3" suffix="back"/>
-    <xacro:arm_z_pole x="0.45" suffix="front"/>
+    <xacro:arm_z_pole x="0.09" suffix="back"/>
+    <xacro:arm_z_pole x="0.24" suffix="front"/>
     <link name="arm_z_pole_endcap">
         <inertial>

File: rosws/src/rover_description/urdf/rover.xacro.urdf (robot description, URDF)
Before this commit: robot rover, 1 links, 0 joints
Links:
- link base_link: geometry collision box size=1 0.5 0.1; visual box size=0.78 0.5 0.1

File: rosws/src/rover_description/urdf/sensors.xacro (robot description, xacro)
@@ -21,5 +21,5 @@
         <parent link="base_link"/>
         <child link="imu_link"/>
-        <origin xyz="0 0 0.125"/>
+        <origin xyz="0 0 0.05"/>
     </joint>
     <gazebo reference="imu_link">
@@ -44,57 +44,3 @@
         </sensor>
     </gazebo>
-    <link name="laser_link">
-        <inertial>
-            <mass value="0.1" />
-            <inertia ixx="0.000115833333333" ixy="0" ixz="0" iyy="0.000115833333333" iyz="0" izz="0.000125" />
-        </inertial>
-        <visual>
-            <origin xyz="0 0 0" rpy="0 0 0" />
-            <geometry>
-                <cylinder radius="0.05" length="0.08" />
-            </geometry>
-        </visual>
-        <collision>
-            <origin xyz="0 0 0" rpy="0 0 0" />
-            <geometry>
-                <cylinder radius="0.05" length="0.08" />
-            </geometry>
-        </collision>
-    </link>
-    <joint name="base_to_laser_link" type="fixed">
-        <parent link="base_link" />
-        <child link="laser_link" />
-        <origin xyz="0 0 0.29" rpy="0 0 0" />
-    </joint>
-    <gazebo reference="laser_link">
-        <sensor type="gpu_ray" name="laser_scanner">
-            <pose>0 0 0.45 1.57 0 0</pose>
-            <visualize>false</visualize>
-            <update_rate>40</update_rate>
-            <ray>
-                <scan>
-                    <horizontal>
-                        <samples>720</samples>
-                        <resolution>0.02</resolution>
-                        <min_angle>-1.57</min_angle>
-                        <max_angle>1.57</max_angle>
-                    </horizontal>
-                </scan>
-                <range>
-                    <min>0.2</min>
-                    <max>30.0</max>
-                    <resolution>0.01</resolution>
-                </range>
-                <noise>
-                    <type>gaussian</type>
-                    <mean>0.0</mean>
-                    <stddev>0.01</stddev>
-                </noise>
-            </ray>
-            <plugin name="gazebo_ros_laser_scan_controller" filename="libgazebo_ros_gpu_laser.so">
-                <topicName>/laser/scan</topicName>
-                <frameName>laser_link</frameName>
-            </plugin>
-        </sensor>
-    </gazebo>
 </robot>

File: rosws/src/rover_description/urdf/stereo.xacro (robot description, xacro)
@@ -23,5 +23,5 @@
         <parent link="base_link"/>
         <child link="stereo_camera_link"/>
-        <origin xyz="0.38 0.1 0.25" rpy="0 0 0"/>
+        <origin xyz="0.38 0.1 0.1" rpy="0 0 0"/>
     </joint>
     <link name="stereo_left_optical_frame"/>

File: rosws/src/rover_description/urdf/wheel.xacro (robot description, xacro)
@@ -1,5 +1,5 @@
 <?xml version="1.0" ?>
 <robot xmlns:xacro="http://www.ros.org/wiki/xacro">
-    <xacro:macro name="wheel" params="suffix attach side">
+    <xacro:macro name="wheel" params="suffix attach side reduction">
         <link name="wheel_leg_${suffix}">
             <inertial>
@@ -8,14 +8,14 @@
             </inertial>
             <visual>
-                <origin xyz="0 0 -0.15" rpy="0 0 0" />
+                <origin xyz="0 0 -0.075" rpy="0 0 0" />
                 <material name="Red" />
                 <geometry>
-                    <cylinder radius="0.1" length="0.3" />
+                    <cylinder radius="0.02" length="0.15" />
                 </geometry>
             </visual>
             <collision>
-                <origin xyz="0 0 -0.15" rpy="0 0 0" />
+                <origin xyz="0 0 -0.075" rpy="0 0 0" />
                 <geometry>
-                    <cylinder radius="0.1" length="0.3" />
+                    <cylinder radius="0.02" length="0.15" />
                 </geometry>
             </collision>
@@ -35,5 +35,5 @@
                 <material name="White" />
                 <geometry>
-                    <cylinder radius="0.1" length="0.1" />
+x                    <cylinder radius="0.1" length="0.1" />
                 </geometry>
             </visual>
@@ -46,5 +46,5 @@
         </link>
         <joint name="leg_to_wheel_${suffix}" type="continuous">
-            <origin xyz="0 ${side * 0.1} -0.3" rpy="0 0 0" />
+            <origin xyz="0 ${side * 0.1} -0.15" rpy="0 0 0" />
             <parent link="wheel_leg_${suffix}" />
             <child link="wheel_${suffix}" />
@@ -75,5 +75,5 @@
             <actuator name="drive_motor_${suffix}">
                 <hardwareInterface>hardware_interface/VelocityJointInterface</hardwareInterface>
-                <mechanicalReduction>1</mechanicalReduction>
+                <mechanicalReduction>${reduction}</mechanicalReduction>
             </actuator>
         </transmission>
