Commit message: more odometry locations, added a laser to the urdf (probably will be unused)
added parameters to the max wheel speed to prepare for fixing proper values for real rover
these values need fixing for actual rover operations

File: rosws/src/rover_description/urdf/sensors.xacro (robot description, xacro)
@@ -94,5 +94,5 @@
                 <topicName>/imu/data</topicName>
                 <serviceName>/imu/service</serviceName>
-                <gaussianNoise>0.05</gaussianNoise>
+                <gaussianNoise>0.0</gaussianNoise>
                 <updateRateHZ>20.0</updateRateHZ>
                 <xyzOffset>0 0 0</xyzOffset>
@@ -103,3 +103,57 @@
         </sensor>
     </gazebo>
+    <link name="laser_link">
+        <inertial>
+            <mass value="0.1" />
+            <inertia ixx="0.000115833333333" ixy="0" ixz="0" iyy="0.000115833333333" iyz="0" izz="0.000125" />
+        </inertial>
+        <visual>
+            <origin xyz="0 0 0" rpy="0 0 0" />
+            <geometry>
+                <cylinder radius="0.05" length="0.08" />
+            </geometry>
+        </visual>
+        <collision>
+            <origin xyz="0 0 0" rpy="0 0 0" />
+            <geometry>
+                <cylinder radius="0.05" length="0.08" />
+            </geometry>
+        </collision>
+    </link>
+    <joint name="base_to_laser_link" type="fixed">
+        <parent link="base_link" />
+        <child link="laser_link" />
+        <origin xyz="0 0 0.29" rpy="0 0 0" />
+    </joint>
+    <gazebo reference="laser_link">
+        <sensor type="gpu_ray" name="laser_scanner">
+            <pose>0 0 0.45 1.57 0 0</pose>
+            <visualize>false</visualize>
+            <update_rate>40</update_rate>
+            <ray>
+                <scan>
+                    <horizontal>
+                        <samples>720</samples>
+                        <resolution>0.02</resolution>
+                        <min_angle>-1.57</min_angle>
+                        <max_angle>1.57</max_angle>
+                    </horizontal>
+                </scan>
+                <range>
+                    <min>0.2</min>
+                    <max>30.0</max>
+                    <resolution>0.01</resolution>
+                </range>
+                <noise>
+                    <type>gaussian</type>
+                    <mean>0.0</mean>
+                    <stddev>0.01</stddev>
+                </noise>
+            </ray>
+            <plugin name="gazebo_ros_laser_scan_controller" filename="libgazebo_ros_gpu_laser.so">
+                <topicName>/laser/scan</topicName>
+                <frameName>laser_link</frameName>
+            </plugin>
+        </sensor>
+    </gazebo>
 </robot>

Commit message: begin code for moveit

File: rosws/src/rover_description/urdf/sensors.xacro (robot description, xacro)
@@ -23,5 +23,5 @@
         <parent link="base_link"/>
         <child link="zed_camera_link"/>
-        <origin xyz="0.38 0.3 0.25" rpy="0 0 0"/>
+        <origin xyz="0.38 0 0.25" rpy="0 0 0"/>
     </joint>
     <gazebo reference="zed_camera_link">

Commit message: start work on new stereo config

File: rosws/src/rover_description/urdf/sensors.xacro (robot description, xacro)
@@ -1,64 +1,5 @@
 <?xml version="1.0" ?>
 <robot xmlns:xacro="http://www.ros.org/wiki/xacro">
-    <link name="zed_camera_link">
-        <inertial>
-            <inertia ixx="0.000604166666667" ixy="0" ixz="0" iyy="0.000166666666667" iyz="0" izz="0.000604166666667"/>
-            <mass value="0.1"/>
-        </inertial>
-        <visual>
-            <material name="Yellow"/>
-            <origin xyz="0 0 0.05" rpy="0 0 0"/>
-            <geometry>
-                <box size="0.1 0.08 0.1"/>
-            </geometry>
-        </visual>
-        <collision>
-            <origin xyz="0 0 0.05" rpy="0 0 0"/>
-            <geometry>
-                <box size="0.1 0.08 0.1"/>
-            </geometry>
-        </collision>
-    </link>
-    <joint name="base_to_camera_link" type="fixed">
-        <parent link="base_link"/>
-        <child link="zed_camera_link"/>
-        <origin xyz="0.38 0 0.25" rpy="0 0 0"/>
-    </joint>
-    <gazebo reference="zed_camera_link">
-        <sensor type="depth" name="zed">
-            <always_on>true</always_on>
-            <update_rate>30</update_rate>
-            <camera>stereo
-                <horizontal_fov>1.65</horizontal_fov>
-                <image>
-                    <format>B8G8R8</format>
-                    <width>1280</width>
-                    <height>720</height>
-                </image>
-                <clip>
-                    <near>0.1</near>
-                    <far>100</far>
-                </clip>
-            </camera>
-            <plugin name="zed_camera_controller" filename="libgazebo_ros_openni_kinect.so">
-                <cameraName>stereo</cameraName>
-                <alwaysOn>true</alwaysOn>
-                <updateRate>15</updateRate>
-                <imageTopicName>left/image_rect_color</imageTopicName>
-                <depthImageTopicName>depth</depthImageTopicName>
-                <pointCloudTopicName>points2</pointCloudTopicName>
-                <cameraInfoTopicName>left/camera_info</cameraInfoTopicName>
-                <depthImageCameraInfoTopicName>depth/camera_info</depthImageCameraInfoTopicName>
-                <frameName>zed_camera_link_optical</frameName>
-                <baseline>0.1</baseline>
-                <distortion_k1>0.0</distortion_k1>
-                <distortion_k2>0.0</distortion_k2>
-                <distortion_k3>0.0</distortion_k3>
-                <distortion_t1>0.0</distortion_t1>
-                <distortion_t2>0.0</distortion_t2>
-                <pointCloudCutoff>0.2</pointCloudCutoff>
-            </plugin>
-        </sensor>
-    </gazebo>
+    <xacro:include filename="stereo.xacro" />
     <link name="imu_link">
         <inertial>

Commit message: Stereo urdf (#12)
* servo test

* change back to victors!

t

* servo test

* change back to victors!

t

* sync

* yay

* ros_control drive

controllers are working, testing of hardware is probably happening on saturday

* docs v. 1

* docs v. 2

* docs v. 2.5

* sumting

* better naming

* test codez

* FOR TESTIJNG

* test2

* test2

* fix idiotic negation

* something

* AMAZING DOCUMENTATION

* moar docs

* bla

* temp

* fix

* what

* start robot_localization

good working odom

* unnessecary codeos

* segment pt1

* start work

* add more stuff to make auton easier

* merge in new teleop

(cherry picked from commit ab3c0ac)

* something yay it kind of works but stupid stuff makes it doesn't

* extra things

* create stereo camera

* sync

* yay

* ros_control drive

controllers are working, testing of hardware is probably happening on saturday

* AMAZING DOCUMENTATION

* moar docs

* temp

* start robot_localization

good working odom

* unnessecary codeos

* segment pt1

* start work

* add more stuff to make auton easier

* servo test

* servo test

* change back to victors!

t

* change back to victors!

t

* sync

* yay

* ros_control drive

controllers are working, testing of hardware is probably happening on saturday

* docs v. 1

* docs v. 2

* docs v. 2.5

* sumting

* better naming

* test codez

* something yay it kind of works but stupid stuff makes it doesn't

* extra things

* fix idiotic negation

* something

* AMAZING DOCUMENTATION

* moar docs

* start work

* merge in new teleop

(cherry picked from commit ab3c0ac)

* Randomized blabla

* yippe yooooooo!

in other words, it functions now

(cherry picked from commit a7708cd)

* pretty much functioning!

* stage 1 of new docs:

add gazebo (As i modified it here)
reformat to make it uniform

* add nav docs

* more odometry locations, added a laser to the urdf (probably will be unused)

added parameters to the max wheel speed to prepare for fixing proper values for real rover
these values need fixing for actual rover operations

* asdf

* calibrate stereo

* change urdf to have similar names to stereo cam

* add disp_to_depth

* make it work with stereo & simulation (hopefully)

* config done for unification

* new cam config

* new cam config

* actually function

* start work on new stereo config

* finish new stereo config (needs testing)

* switch sim back over to stereo...

* fix urdf for stereo cameras

* new

File: rosws/src/rover_description/urdf/sensors.xacro (robot description, xacro)
@@ -1,68 +1,9 @@
 <?xml version="1.0" ?>
 <robot xmlns:xacro="http://www.ros.org/wiki/xacro">
-    <link name="zed_camera_link">
-        <inertial>
-            <inertia ixx="0.000604166666667" ixy="0" ixz="0" iyy="0.000166666666667" iyz="0" izz="0.000604166666667"/>
-            <mass value="0.1"/>
-        </inertial>
-        <visual>
-            <material name="Yellow"/>
-            <origin xyz="0 0 0.05" rpy="0 0 0"/>
-            <geometry>
-                <box size="0.1 0.08 0.1"/>
-            </geometry>
-        </visual>
-        <collision>
-            <origin xyz="0 0 0.05" rpy="0 0 0"/>
-            <geometry>
-                <box size="0.1 0.08 0.1"/>
-            </geometry>
-        </collision>
-    </link>
-    <joint name="base_to_camera_link" type="fixed">
-        <parent link="base_link"/>
-        <child link="zed_camera_link"/>
-        <origin xyz="0.38 0 0.25" rpy="0 0 0"/>
-    </joint>
-    <gazebo reference="zed_camera_link">
-        <sensor type="depth" name="zed">
-            <always_on>true</always_on>
-            <update_rate>30</update_rate>
-            <camera>stereo
-                <horizontal_fov>1.65</horizontal_fov>
-                <image>
-                    <format>B8G8R8</format>
-                    <width>1280</width>
-                    <height>720</height>
-                </image>
-                <clip>
-                    <near>0.1</near>
-                    <far>100</far>
-                </clip>
-            </camera>
-            <plugin name="zed_camera_controller" filename="libgazebo_ros_openni_kinect.so">
-                <cameraName>zed</cameraName>
-                <alwaysOn>true</alwaysOn>
-                <updateRate>15</updateRate>
-                <imageTopicName>rgb/image_raw</imageTopicName>
-                <depthImageTopicName>depth/image_raw</depthImageTopicName>
-                <pointCloudTopicName>points</pointCloudTopicName>
-                <cameraInfoTopicName>rgb/camera_info</cameraInfoTopicName>
-                <depthImageCameraInfoTopicName>depth/camera_info</depthImageCameraInfoTopicName>
-                <frameName>zed_camera_link_optical</frameName>
-                <baseline>0.1</baseline>
-                <distortion_k1>0.0</distortion_k1>
-                <distortion_k2>0.0</distortion_k2>
-                <distortion_k3>0.0</distortion_k3>
-                <distortion_t1>0.0</distortion_t1>
-                <distortion_t2>0.0</distortion_t2>
-                <pointCloudCutoff>0.2</pointCloudCutoff>
-            </plugin>
-        </sensor>
-    </gazebo>
+    <xacro:include filename="stereo.xacro" />
     <link name="imu_link">
         <inertial>
             <inertia ixx="0.000604166666667" ixy="0" ixz="0" iyy="0.000166666666667" iyz="0" izz="0.000604166666667"/>
-            <mass value="0.1"/>
+            <mass value="0.05"/>
         </inertial>
         <visual>
@@ -78,24 +19,81 @@
     </link>
     <joint name="base_to_imu_link" type="fixed">
-        <parent link="base_link" />
-        <child link="imu_link" />
-        <origin xyz="0 0 0.125" />
+        <parent link="base_link"/>
+        <child link="imu_link"/>
+        <origin xyz="0 0 0.125"/>
     </joint>
     <gazebo reference="imu_link">
+        <gravity>true</gravity>
         <sensor name="imu_sensor" type="imu">
-            <always_on>1</always_on>
-            <update_rate>250</update_rate>
+            <always_on>true</always_on>
+            <update_rate>100</update_rate>
+            <visualize>true</visualize>
             <topic>__default_topic__</topic>
-            <imu />
             <plugin name="imu_plugin" filename="libgazebo_ros_imu_sensor.so">
-                <topicName>imu/data</topicName>
+                <alwaysOn>true</alwaysOn>
                 <bodyName>imu_link</bodyName>
-                <frameName>imu_link</frameName>
-                <updateRateHZ>250</updateRateHZ>
+                <topicName>/imu/data</topicName>
+                <serviceName>/imu/service</serviceName>
                 <gaussianNoise>0.0</gaussianNoise>
+                <updateRateHZ>20.0</updateRateHZ>
                 <xyzOffset>0 0 0</xyzOffset>
                 <rpyOffset>0 0 0</rpyOffset>
+                <frameName>imu_link</frameName>
             </plugin>
-            <pose>0 0 0 0 0 0</pose>
+            <pose>0 0 0 0 0 0</pose> <!-- todo: make sure this is right -->
+        </sensor>
+    </gazebo>
+    <link name="laser_link">
+        <inertial>
+            <mass value="0.1" />
+            <inertia ixx="0.000115833333333" ixy="0" ixz="0" iyy="0.000115833333333" iyz="0" izz="0.000125" />
+        </inertial>
+        <visual>
+            <origin xyz="0 0 0" rpy="0 0 0" />
+            <geometry>
+                <cylinder radius="0.05" length="0.08" />
+            </geometry>
+        </visual>
+        <collision>
+            <origin xyz="0 0 0" rpy="0 0 0" />
+            <geometry>
+                <cylinder radius="0.05" length="0.08" />
+            </geometry>
+        </collision>
+    </link>
+    <joint name="base_to_laser_link" type="fixed">
+        <parent link="base_link" />
+        <child link="laser_link" />
+        <origin xyz="0 0 0.29" rpy="0 0 0" />
+    </joint>
+    <gazebo reference="laser_link">
+        <sensor type="gpu_ray" name="laser_scanner">
+            <pose>0 0 0.45 1.57 0 0</pose>
+            <visualize>false</visualize>
+            <update_rate>40</update_rate>
+            <ray>
+                <scan>
+                    <horizontal>
+                        <samples>720</samples>
+                        <resolution>0.02</resolution>
+                        <min_angle>-1.57</min_angle>
+                        <max_angle>1.57</max_angle>
+                    </horizontal>
+                </scan>
+                <range>
+                    <min>0.2</min>
+                    <max>30.0</max>
+                    <resolution>0.01</resolution>
+                </range>
+                <noise>
+                    <type>gaussian</type>
+                    <mean>0.0</mean>
+                    <stddev>0.01</stddev>
+                </noise>
+            </ray>
+            <plugin name="gazebo_ros_laser_scan_controller" filename="libgazebo_ros_gpu_laser.so">
+                <topicName>/laser/scan</topicName>
+                <frameName>laser_link</frameName>
+            </plugin>
         </sensor>
     </gazebo>

File: rosws/src/rover_description/urdf/wheel.xacro (robot description, xacro)
@@ -28,5 +28,5 @@
         <link name="wheel_${suffix}">
             <inertial>
-                <mass value="1" />
+                <mass value="0.25" />
                 <inertia ixx="0.00333333333333" ixy="0" ixz="0" iyy="0.005" iyz="0" izz="0.00333333333333" />
             </inertial>
@@ -50,5 +50,5 @@
             <child link="wheel_${suffix}" />
             <axis xyz="0 1 0" />
-            <dynamics damping="0.015" friction="0.02" />
+            <!-- dynamics damping="0.015" friction="0.02" / -->
         </joint>
         <gazebo reference="wheel_leg_${suffix}">

Commit message: update imu posistion

File: rosws/src/rover_description/urdf/sensors.xacro (robot description, xacro)
@@ -21,5 +21,5 @@
         <parent link="base_link"/>
         <child link="imu_link"/>
-        <origin xyz="0 0 0.05"/>
+        <origin xyz="0.2 0 0.1"/>
     </joint>
     <gazebo reference="imu_link">
