Commit message: begin science arm

File: rosws/src/rover_description/urdf/grippers/science_gripper.xacro (robot description, xacro)
@@ -3,6 +3,6 @@
     <link name="science_drill">
         <inertial>
-            <mass value="1.0"/>
-            <inertia ixx="0.00536962333333" ixy="0" ixz="0" iyy="0.00536962333333" iyz="0" izz="0.00032258"/>
+            <mass value="0.15"/>
+            <inertia ixx="0.000186048375" ixy="0" ixz="0" iyy="0.000186048375" iyz="0" izz="1.209675e-05" />
         </inertial>
         <visual>
@@ -63,4 +63,6 @@
         <origin xyz="0.14 0 0" rpy="0 0 0" />
         <axis xyz="0 0 1" />
+        <dynamics friction="0" damping="0.02" />
+        <limit effort="250" velocity="0.3" lower="-100000000000" upper="1000000000000"/>
     </joint>
     <joint name="arm_inner_to_science_sensors_crossbar" type="fixed">

Commit message: tune pids better

File: rosws/src/rover_description/urdf/grippers/science_gripper.xacro (robot description, xacro)
@@ -76,5 +76,5 @@
         <origin xyz="0 -0.05968 0" rpy="0 0 0" />
         <axis xyz="0 0 1" />
-        <limit effort="2000" velocity="1" lower="0" upper="0.23"/>
+        <limit effort="2000" velocity="1" lower="0" upper="0.25"/>
     </joint>
     <transmission name="science_drill_trans">
