Commit message: add science gripper

File: rosws/src/rover_description/urdf/grippers/normal_gripper.xacro (robot description, xacro)
@@ -23,5 +23,5 @@
         <inertial>
             <mass value="0.05" />
-            <inertia ixx="1.29032e-05" ixy="0" ixz="0" iyy="0.0005127016" iyz="0" izz="0.0005127016" />
+            <inertia ixx="4.94791666667e-05" ixy="0" ixz="0" iyy="4.94791666667e-05" iyz="0" izz="1.5625e-05" />
         </inertial>
         <collision>

Commit message: fuckit 2: electric boogaloo

File: rosws/src/rover_description/urdf/grippers/normal_gripper.xacro (robot description, xacro)
@@ -25,38 +25,65 @@
         </visual>
     </link>
-    <link name="grip_spin">
+    <link name="grip_tilt">
         <inertial>
-            <mass value="0.05" />
-            <inertia ixx="4.94791666667e-05" ixy="0" ixz="0" iyy="4.94791666667e-05" iyz="0" izz="1.5625e-05" />
+            <mass value="0.2" />
+            <inertia ixx="3.65666666667e-05" ixy="0" ixz="0" iyy="0.000137816666667" iyz="0" izz="0.00016875" />
         </inertial>
         <collision>
-            <origin xyz="0 0 -0.05" rpy="0 0 0" />
+            <origin xyz="0.045 0 0" rpy="0 0 0" />
             <geometry>
-                <cylinder radius="0.025" length="0.1" />
+                <box size="0.09 0.045 0.013" />
             </geometry>
         </collision>
         <visual>
             <material name="Blue" />
-            <origin xyz="0 0 -0.05" rpy="0 0 0" />
+            <origin xyz="0.045 0 0" rpy="0 0 0" />
             <geometry>
-                <cylinder radius="0.025" length="0.1" />
+                <box size="0.09 0.045 0.013" />
             </geometry>
         </visual>
     </link>
-    <joint name="arm_outer_to_grip_spin" type="continuous">
+    <link name="grip_spin">
+        <inertial>
+            <mass value="0.05" />
+            <inertia ixx="1.46e-05" ixy="0" ixz="0" iyy="1.46e-05" iyz="0" izz="2.89e-05" />
+        </inertial>
+        <collision>
+            <origin xyz="0 0 0.003" rpy="0 0 0"/>
+            <geometry>
+                <cylinder radius="0.034" length="0.006" />
+            </geometry>
+        </collision>
+        <visual>
+            <origin xyz="0 0 0.003" rpy="0 0 0"/>
+            <geometry>
+                <cylinder radius="0.034" length="0.006" />
+            </geometry>
+        </visual>
+    </link>
+    <joint name="arm_outer_to_grip_tilt" type="revolute">
         <parent link="arm_outer" />
-        <child link="grip_spin" />
-        <origin xyz="0.225 0 -0.0127" rpy="0 0 0" />
-        <axis xyz="0 0 1" />
+        <child link="grip_tilt" />
+        <origin xyz="0.225 0 0" rpy="0 0 0" />
+        <axis xyz="1 0 0" />
+        <limit upper="1.57" lower="-1.04" effort="300" velocity="0.3"/>
     </joint>
-    <joint name="arm_inner_to_arm_outer" type="continuous">
+    <joint name="arm_inner_to_arm_outer" type="revolute">
         <parent link="arm_inner" />
         <child link="arm_outer" />
         <origin xyz="0.217 0 -0.038" rpy="0 0 0" />
         <axis xyz="0 0 1" />
+        <limit upper="1.57" lower="-1.57" effort="500" velocity="0.8" />
+    </joint>
+    <joint name="grip_tilt_to_grip_spin" type="revolute">
+        <parent link="grip_tilt" />
+        <child link="grip_spin" />
+        <origin xyz="0.09 0 -0.0065" rpy="0 0 0" />
+        <axis xyz="0 0 1" />
+        <limit upper="12.4" lower="-12.4" effort="400" velocity="1" />
     </joint>
     <transmission name="arm_sping">
         <type>transmission_interface/SimpleTransmission</type>
-        <joint name="arm_outer_to_grip_spin">
+        <joint name="arm_outer_to_grip_tilt">
             <hardwareInterface>hardware_interface/EffortJointInterface</hardwareInterface>
         </joint>
@@ -64,4 +91,14 @@
             <hardwareInterface>hardware_interface/EffortJointInterface</hardwareInterface>
             <mechanicalReduction>-6.33333333</mechanicalReduction>
+        </actuator>
+    </transmission>
+    <transmission name="arm_spingt">
+        <type>transmission_interface/SimpleTransmission</type>
+        <joint name="grip_tilt_to_grip_spin">
+            <hardwareInterface>hardware_interface/EffortJointInterface</hardwareInterface>
+        </joint>
+        <actuator name="arm_spin_outer_motor">
+            <hardwareInterface>hardware_interface/EffortJointInterface</hardwareInterface>
+            <mechanicalReduction>-5.25</mechanicalReduction>
         </actuator>
     </transmission>
@@ -76,3 +113,67 @@
         </actuator>
     </transmission>
+    <xacro:macro name="tooth" params="offsetx offsety rotang suffix">
+        <link name="tooth_${suffix}_upper">
+            <inertial>
+                <mass value="0.3" />
+                <inertia ixx="3.4e-06" ixy="0" ixz="0" iyy="6.5e-05" iyz="0" izz="6.34e-05" />
+            </inertial>
+            <collision>
+                <origin xyz="0.025 0 0" rpy="0 0.2 0" />
+                <geometry>
+                    <box size="0.05 0.006 0.01" />
+                </geometry>
+            </collision>
+            <visual>
+                <origin xyz="0.025 0 0" rpy="0 0.2 0" />
+                <geometry>
+                    <box size="0.05 0.006 0.01" />
+                </geometry>
+            </visual>
+        </link>
+        <link name="tooth_${suffix}_lower">
+            <inertial>
+                <mass value="0.3" />
+                <inertia ixx="3.4e-06" ixy="0" ixz="0" iyy="6.5e-05" iyz="0" izz="6.34e-05" />
+            </inertial>
+            <collision>
+                <origin xyz="0.025 0 0" rpy="0 0 0" />
+                <geometry>
+                    <box size="0.05 0.006 0.01" />
+                </geometry>
+            </collision>
+            <visual>
+                <origin xyz="0.025 0 0" rpy="0 0 0" />
+                <geometry>
+                    <box size="0.05 0.006 0.01" />
+                </geometry>
+            </visual>
+        </link>
+        <joint name="grip_spin_to_tooth_${suffix}" type="revolute">
+            <parent link="grip_spin" />
+            <child link="tooth_${suffix}_upper" />
+            <origin xyz="${offsetx} ${offsety} -0.006" rpy="0 0 ${rotang}" />
+            <limit upper="1.16" lower="0" effort="400" velocity="0.3" />
+            <axis xyz="0 1 0" />
+        </joint>
+        <joint name="tooth_${suffix}_upper_to_lower" type="fixed">
+            <parent link="tooth_${suffix}_upper" />
+            <child link="tooth_${suffix}_lower" />
+            <origin xyz="0.05 0 -0.005" rpy="0 0.69 0" />
+        </joint>
+        <transmission name="arm_tooth_${suffix}">
+            <type>transmission_interface/SimpleTransmission</type>
+            <joint name="grip_spin_to_tooth_${suffix}">
+                <hardwareInterface>hardware_interface/EffortJointInterface</hardwareInterface>
+            </joint>
+            <actuator name="motor_tooth_${suffix}">
+                <hardwareInterface>hardware_interface/EffortJointInterface</hardwareInterface>
+                <mechanicalReduction>-10</mechanicalReduction>
+            </actuator>
+        </transmission>
+    </xacro:macro>
+    <xacro:tooth offsetx="0.0194" offsety="0.0057" rotang="0" suffix="front" />
+    <xacro:tooth offsetx="0.0057" offsety="0.0194" rotang="1.57" suffix="left" />
+    <xacro:tooth offsetx="-0.0194" offsety="0.0057" rotang="3.14" suffix="rear" />
+    <xacro:tooth offsetx="-0.0057" offsety="-0.0194" rotang="4.71" suffix="right" />
 </robot>

Commit message: it works?

File: rosws/src/rover_description/urdf/grippers/normal_gripper.xacro (robot description, xacro)
@@ -66,5 +66,5 @@
         <child link="grip_tilt" />
         <origin xyz="0.225 0 0" rpy="0 0 0" />
-        <axis xyz="1 0 0" />
+        <axis xyz="0 1 0" />
         <limit upper="1.57" lower="-1.04" effort="300" velocity="0.3"/>
     </joint>

Commit message: Arm software (#16)
* Start new arm

including new stars like:

   - the poles
   - the box
   - the encap

and returning players like:

   - the gripper

* new ARM!!!!!

* better naming

* move eml_uberdriver

* almost done docs for eml_uberdriver

WARNING: this will probably get moved out to rtd for a seperate system, but for now
it is staying here

* fix uberfirmware

* START ARM

* begin work on rover arm,

* more arm

* stuff in progress

* current version

* asdf

* reformat arm to a better format

* add science gripper

* add science controllers

* reorg arm_hw

* begin science arm

* more arm

* tune pids better

* begin as

* asdf - asdf

* add various things

* change outdoor_world to support multiple grippers

a sane commit message?

* further change

* start work on new arm software

for test

it'll work
i promise
no i dont
neveer mind

* maybe working code for arm

* changed the address to match hardware

* stop spamming a you git

* modify

GABE WHY

* yayyayayayaya

why am i so tired

* add motor constants

* hmmmm

* 2 is not wired?

* HUZZAH (it works)

this is a matthew commit, under gabe's account(maybe)

* last minute changes

* fuckit 2: electric boogaloo

* it works?

* add gripper

* remove

* dd more debugs

* woopee

* woopee

* fixed drive constants

* stuff??

* adf

* ASDF

* please stop annoying me

* asdf

File: rosws/src/rover_description/urdf/grippers/normal_gripper.xacro (robot description, xacro)
@@ -25,38 +25,65 @@
         </visual>
     </link>
-    <link name="grip_spin">
+    <link name="grip_tilt">
         <inertial>
-            <mass value="0.05" />
-            <inertia ixx="4.94791666667e-05" ixy="0" ixz="0" iyy="4.94791666667e-05" iyz="0" izz="1.5625e-05" />
+            <mass value="0.2" />
+            <inertia ixx="3.65666666667e-05" ixy="0" ixz="0" iyy="0.000137816666667" iyz="0" izz="0.00016875" />
         </inertial>
         <collision>
-            <origin xyz="0 0 -0.05" rpy="0 0 0" />
+            <origin xyz="0.045 0 0" rpy="0 0 0" />
             <geometry>
-                <cylinder radius="0.025" length="0.1" />
+                <box size="0.09 0.045 0.013" />
             </geometry>
         </collision>
         <visual>
             <material name="Blue" />
-            <origin xyz="0 0 -0.05" rpy="0 0 0" />
+            <origin xyz="0.045 0 0" rpy="0 0 0" />
             <geometry>
-                <cylinder radius="0.025" length="0.1" />
+                <box size="0.09 0.045 0.013" />
             </geometry>
         </visual>
     </link>
-    <joint name="arm_outer_to_grip_spin" type="continuous">
+    <link name="grip_spin">
+        <inertial>
+            <mass value="0.05" />
+            <inertia ixx="1.46e-05" ixy="0" ixz="0" iyy="1.46e-05" iyz="0" izz="2.89e-05" />
+        </inertial>
+        <collision>
+            <origin xyz="0 0 0.003" rpy="0 0 0"/>
+            <geometry>
+                <cylinder radius="0.034" length="0.006" />
+            </geometry>
+        </collision>
+        <visual>
+            <origin xyz="0 0 0.003" rpy="0 0 0"/>
+            <geometry>
+                <cylinder radius="0.034" length="0.006" />
+            </geometry>
+        </visual>
+    </link>
+    <joint name="arm_outer_to_grip_tilt" type="revolute">
         <parent link="arm_outer" />
-        <child link="grip_spin" />
-        <origin xyz="0.225 0 -0.0127" rpy="0 0 0" />
-        <axis xyz="0 0 1" />
+        <child link="grip_tilt" />
+        <origin xyz="0.225 0 0" rpy="0 0 0" />
+        <axis xyz="0 1 0" />
+        <limit upper="1.57" lower="-1.04" effort="300" velocity="0.3"/>
     </joint>
-    <joint name="arm_inner_to_arm_outer" type="continuous">
+    <joint name="arm_inner_to_arm_outer" type="revolute">
         <parent link="arm_inner" />
         <child link="arm_outer" />
         <origin xyz="0.217 0 -0.038" rpy="0 0 0" />
         <axis xyz="0 0 1" />
+        <limit upper="1.57" lower="-1.57" effort="500" velocity="0.8" />
+    </joint>
+    <joint name="grip_tilt_to_grip_spin" type="revolute">
+        <parent link="grip_tilt" />
+        <child link="grip_spin" />
+        <origin xyz="0.09 0 -0.0065" rpy="0 0 0" />
+        <axis xyz="0 0 1" />
+        <limit upper="12.4" lower="-12.4" effort="400" velocity="1" />
     </joint>
     <transmission name="arm_sping">
         <type>transmission_interface/SimpleTransmission</type>
-        <joint name="arm_outer_to_grip_spin">
+        <joint name="arm_outer_to_grip_tilt">
             <hardwareInterface>hardware_interface/EffortJointInterface</hardwareInterface>
         </joint>
@@ -64,4 +91,14 @@
             <hardwareInterface>hardware_interface/EffortJointInterface</hardwareInterface>
             <mechanicalReduction>-6.33333333</mechanicalReduction>
+        </actuator>
+    </transmission>
+    <transmission name="arm_spingt">
+        <type>transmission_interface/SimpleTransmission</type>
+        <joint name="grip_tilt_to_grip_spin">
+            <hardwareInterface>hardware_interface/EffortJointInterface</hardwareInterface>
+        </joint>
+        <actuator name="arm_spin_outer_motor">
+            <hardwareInterface>hardware_interface/EffortJointInterface</hardwareInterface>
+            <mechanicalReduction>-5.25</mechanicalReduction>
         </actuator>
     </transmission>
@@ -76,3 +113,67 @@
         </actuator>
     </transmission>
+    <xacro:macro name="tooth" params="offsetx offsety rotang suffix">
+        <link name="tooth_${suffix}_upper">
+            <inertial>
+                <mass value="0.3" />
+                <inertia ixx="3.4e-06" ixy="0" ixz="0" iyy="6.5e-05" iyz="0" izz="6.34e-05" />
+            </inertial>
+            <collision>
+                <origin xyz="0.025 0 0" rpy="0 0.2 0" />
+                <geometry>
+                    <box size="0.05 0.006 0.01" />
+                </geometry>
+            </collision>
+            <visual>
+                <origin xyz="0.025 0 0" rpy="0 0.2 0" />
+                <geometry>
+                    <box size="0.05 0.006 0.01" />
+                </geometry>
+            </visual>
+        </link>
+        <link name="tooth_${suffix}_lower">
+            <inertial>
+                <mass value="0.3" />
+                <inertia ixx="3.4e-06" ixy="0" ixz="0" iyy="6.5e-05" iyz="0" izz="6.34e-05" />
+            </inertial>
+            <collision>
+                <origin xyz="0.025 0 0" rpy="0 0 0" />
+                <geometry>
+                    <box size="0.05 0.006 0.01" />
+                </geometry>
+            </collision>
+            <visual>
+                <origin xyz="0.025 0 0" rpy="0 0 0" />
+                <geometry>
+                    <box size="0.05 0.006 0.01" />
+                </geometry>
+            </visual>
+        </link>
+        <joint name="grip_spin_to_tooth_${suffix}" type="revolute">
+            <parent link="grip_spin" />
+            <child link="tooth_${suffix}_upper" />
+            <origin xyz="${offsetx} ${offsety} -0.006" rpy="0 0 ${rotang}" />
+            <limit upper="1.16" lower="0" effort="400" velocity="0.3" />
+            <axis xyz="0 1 0" />
+        </joint>
+        <joint name="tooth_${suffix}_upper_to_lower" type="fixed">
+            <parent link="tooth_${suffix}_upper" />
+            <child link="tooth_${suffix}_lower" />
+            <origin xyz="0.05 0 -0.005" rpy="0 0.69 0" />
+        </joint>
+        <transmission name="arm_tooth_${suffix}">
+            <type>transmission_interface/SimpleTransmission</type>
+            <joint name="grip_spin_to_tooth_${suffix}">
+                <hardwareInterface>hardware_interface/EffortJointInterface</hardwareInterface>
+            </joint>
+            <actuator name="motor_tooth_${suffix}">
+                <hardwareInterface>hardware_interface/EffortJointInterface</hardwareInterface>
+                <mechanicalReduction>-1</mechanicalReduction>
+            </actuator>
+        </transmission>
+    </xacro:macro>
+    <xacro:tooth offsetx="0.0194" offsety="0.0057" rotang="0" suffix="front" />
+    <xacro:tooth offsetx="0.0057" offsety="0.0194" rotang="1.57" suffix="left" />
+    <xacro:tooth offsetx="-0.0194" offsety="0.0057" rotang="3.14" suffix="rear" />
+    <xacro:tooth offsetx="-0.0057" offsety="-0.0194" rotang="4.71" suffix="right" />
 </robot>
