File: pcbs/science_boards/ScienceDuino.brd (EAGLE design)
At the start: 160 x 100 mm, 18 parts, among them X1 Barometer, X10 5566-2, X2 Anemometer, X3 EC, X4 EC-Temperature, X5 PH, X6 Temperature+Humidity, X7 Hydrogen, X8 Geiger counter, X9 Dust sensor

Commit message: I hate hamza 2
Connections:
- new net 7V: X2.3
- net DATA1_ECT: now also A1.8; no longer A1.5
- net DATA1_GEI: now also A1.5; no longer A1.8
- net VCC: no longer X2.3
Changed lines of the file:
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@@
 <?xml version="1.0" encoding="utf-8"?>
 <!DOCTYPE eagle SYSTEM "eagle.dtd">
-<eagle version="8.6.0">
+<eagle version="8.6.3">
 <drawing>
 <settings>
@@
 <contactref element="X1" pad="3"/>
 <contactref element="A1" pad="27"/>
-<contactref element="X2" pad="3"/>
 <contactref element="X3" pad="3"/>
 <contactref element="X4" pad="3"/>
@@
 <wire x1="-38.1" y1="99.06" x2="-26.67" y2="99.06" width="0" layer="19" extent="1-1"/>
 <wire x1="-53.34" y1="100.33" x2="-38.1" y2="99.06" width="0" layer="19" extent="1-1"/>
-<wire x1="-19.49" y1="73.87" x2="-19.49" y2="90.38" width="0" layer="19" extent="1-1"/>
-<wire x1="-20.76" y1="57.36" x2="-19.49" y2="73.87" width="0" layer="19" extent="1-1"/>
-<wire x1="-37.27" y1="73.87" x2="-19.49" y2="73.87" width="0" layer="19" extent="1-1"/>
+<wire x1="-54.61" y1="82.55" x2="-53.34" y2="100.33" width="0" layer="19" extent="1-1"/>
+<wire x1="-55.05" y1="73.87" x2="-54.61" y2="82.55" width="0" layer="19" extent="1-1"/>
+<wire x1="-56.32" y1="57.36" x2="-55.05" y2="73.87" width="0" layer="19" extent="1-1"/>
+<wire x1="-37.27" y1="73.87" x2="-55.05" y2="73.87" width="0" layer="19" extent="1-1"/>
 <wire x1="-38.54" y1="57.36" x2="-37.27" y2="73.87" width="0" layer="19" extent="1-1"/>
-<wire x1="-55.05" y1="73.87" x2="-37.27" y2="73.87" width="0" layer="19" extent="1-1"/>
-<wire x1="-54.61" y1="82.55" x2="-55.05" y2="73.87" width="0" layer="19" extent="1-1"/>
-<wire x1="-56.32" y1="57.36" x2="-55.05" y2="73.87" width="0" layer="19" extent="1-1"/>
+<wire x1="-20.76" y1="57.36" x2="-38.54" y2="57.36" width="0" layer="19" extent="1-1"/>
 <wire x1="-72.83" y1="73.87" x2="-55.05" y2="73.87" width="0" layer="19" extent="1-1"/>
 <wire x1="-76.2" y1="82.55" x2="-72.83" y2="73.87" width="0" layer="19" extent="1-1"/>
@@
 <signal name="DATA1_ECT">
 <contactref element="X4" pad="1"/>
-<contactref element="A1" pad="5"/>
-<wire x1="-30.48" y1="33.02" x2="-20.76" y2="51.86" width="0" layer="19" extent="1-1"/>
+<contactref element="A1" pad="8"/>
+<wire x1="-30.48" y1="25.4" x2="-20.76" y2="51.86" width="0" layer="19" extent="1-1"/>
 </signal>
 <signal name="DATA1_HY">
@@
 <signal name="DATA1_GEI">
 <contactref element="X8" pad="1"/>
-<contactref element="A1" pad="8"/>
-<wire x1="-30.48" y1="25.4" x2="-38.54" y2="51.86" width="0" layer="19" extent="1-1"/>
+<contactref element="A1" pad="5"/>
+<wire x1="-30.48" y1="33.02" x2="-38.54" y2="51.86" width="0" layer="19" extent="1-1"/>
 </signal>
 <signal name="DO_RX">
@@
 <wire x1="-30.48" y1="22.86" x2="-23.69" y2="84.88" width="0" layer="19" extent="1-1"/>
 </signal>
+<signal name="7V">
+<contactref element="X2" pad="3"/>
+</signal>
 </signals>
