File: pcbs/science_boards/ScienceDuino.sch (EAGLE design)
At the start: 18 parts, among them X1 Barometer, X10 5566-2, X2 Anemometer, X3 EC, X4 EC-Temperature, X5 PH, X6 Temperature+Humidity, X7 Hydrogen, X8 Geiger counter, X9 Dust sensor

Commit message: I hate hamza 2
Connections:
- new net 7V: X2-3.S
- net DATA1_ECT: now also A1.D5; no longer A1.D2
- net DATA1_GEI: now also A1.D2; no longer A1.D5
- net VCC: no longer X2-3.S
Changed lines of the file:
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@@
 <?xml version="1.0" encoding="utf-8"?>
 <!DOCTYPE eagle SYSTEM "eagle.dtd">
-<eagle version="8.6.0">
+<eagle version="8.6.3">
 <drawing>
 <settings>
@@
 </segment>
 <segment>
-<pinref part="X2" gate="-3" pin="S"/>
-<wire x1="-7.62" y1="68.58" x2="-22.86" y2="68.58" width="0.1524" layer="91"/>
-<label x="-22.86" y="68.58" size="1.778" layer="95"/>
-</segment>
-<segment>
 <pinref part="X3" gate="-3" pin="S"/>
 <wire x1="-7.62" y1="53.34" x2="-22.86" y2="53.34" width="0.1524" layer="91"/>
@@
 </segment>
 <segment>
-<pinref part="A1" gate="G$1" pin="D2"/>
-<wire x1="30.48" y1="68.58" x2="15.24" y2="68.58" width="0.1524" layer="91"/>
-<label x="15.24" y="68.58" size="1.778" layer="95"/>
+<pinref part="A1" gate="G$1" pin="D5"/>
+<wire x1="30.48" y1="60.96" x2="15.24" y2="60.96" width="0.1524" layer="91"/>
+<label x="15.24" y="60.96" size="1.778" layer="95"/>
 </segment>
 </net>
@@
 </segment>
 <segment>
-<pinref part="A1" gate="G$1" pin="D5"/>
-<wire x1="30.48" y1="60.96" x2="15.24" y2="60.96" width="0.1524" layer="91"/>
-<label x="15.24" y="60.96" size="1.778" layer="95"/>
+<pinref part="A1" gate="G$1" pin="D2"/>
+<wire x1="30.48" y1="68.58" x2="15.24" y2="68.58" width="0.1524" layer="91"/>
+<label x="15.24" y="68.58" size="1.778" layer="95"/>
 </segment>
 </net>
@@
 </segment>
 </net>
+<net name="7V" class="0">
+<segment>
+<pinref part="X2" gate="-3" pin="S"/>
+<wire x1="-7.62" y1="68.58" x2="-22.86" y2="68.58" width="0.1524" layer="91"/>
+<label x="-22.86" y="68.58" size="1.778" layer="95"/>
+</segment>
+</net>

Commit message: i2c stuff
Parts:
- added C7, C8, C9: (no value), rcl:C-USC1206
- added Q1: BSS138, bss138_10:BSS138
- added R13, R14: 10k, rcl:R-US_R1206
Connections:
- net 7V renamed +7V
- new net 3.3: Q1.G, R13.2
- new net SCL_HV: Q1.D, R14.1
- net GND: now also C7.2, C8.2, C9.2
- net SCL: now also Q1.S, R13.1
- net VCC: now also C7.1, C8.1, C9.1
Other:
- moved on the sheet: R1, SV1, SV2, SV3, SV4, SV5, X1-1, X1-2, X1-3, X1-4, X10-1, X10-2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
