File: pcbs/Battery PCBS/Battery Checker.sch (EAGLE design)
At the start: 19 parts

Commit message: added logic level converter
Parts:
- added BATTERY_CON_2: (no value), con-phoenix-254:MPT4
- added Q1, Q2: BSS138, bss138_10:BSS138
- added R13, R14, R15, R16: 10k, rcl:R-US_R1206
Connections:
- new net 3.3: Q1.G, Q2.G, R13.2, R15.2, U$1.3.3V
- new net SCL_HV: Q1.D, R14.1, U$1.A5
- new net SDA_HV: Q2.D, R16.1, U$1.A4
- net BATT2: now also BATTERY_CON_2-1.1
- net BATT3: now also BATTERY_CON_2-2.1
- net BATT4: now also BATTERY_CON_2-3.1
- net BATT5: now also BATTERY_CON_2-4.1
- net SCL: now also Q1.S, R13.1; no longer U$1.A5
- net SDA: now also Q2.S, R15.1; no longer U$1.A4
- net VIN: now also R14.2, R16.2
Changed lines of the file:
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@@
 <setting verticaltext="up"/>
 </settings>
-<grid distance="0.1" unitdist="inch" unit="inch" style="lines" multiple="1" display="yes" altdistance="0.01" altunitdist="inch" altunit="inch"/>
+<grid distance="0.1" unitdist="inch" unit="inch" style="lines" multiple="1" display="no" altdistance="0.01" altunitdist="inch" altunit="inch"/>
 <layers>
 <layer number="1" name="Top" color="4" fill="1" visible="no" active="no"/>
@@
 <layer number="97" name="Info" color="7" fill="1" visible="yes" active="yes"/>
 <layer number="98" name="Guide" color="6" fill="1" visible="yes" active="yes"/>
+<layer number="99" name="SpiceOrder" color="5" fill="1" visible="no" active="no"/>
 </layers>
 <schematic xreflabel="%F%N/%S.%C%R" xrefpart="/%S.%C%R">
@@
 <part name="R12" library="rcl" library_urn="urn:adsk.eagle:library:334" deviceset="R-US_" device="R1206" package3d_urn="urn:adsk.eagle:package:23540/2" value="10k"/>
 <part name="SUPPLY5" library="supply2" library_urn="urn:adsk.eagle:library:372" deviceset="GND" device=""/>
+<part name="Q1" library="bss138_10" deviceset="BSS138" device=""/>
+<part name="Q2" library="bss138_10" deviceset="BSS138" device=""/>
+<part name="R13" library="rcl" library_urn="urn:adsk.eagle:library:334" deviceset="R-US_" device="R1206" package3d_urn="urn:adsk.eagle:package:23540/2" value="10k"/>
+<part name="R14" library="rcl" library_urn="urn:adsk.eagle:library:334" deviceset="R-US_" device="R1206" package3d_urn="urn:adsk.eagle:package:23540/2" value="10k"/>
+<part name="R15" library="rcl" library_urn="urn:adsk.eagle:library:334" deviceset="R-US_" device="R1206" package3d_urn="urn:adsk.eagle:package:23540/2" value="10k"/>
+<part name="R16" library="rcl" library_urn="urn:adsk.eagle:library:334" deviceset="R-US_" device="R1206" package3d_urn="urn:adsk.eagle:package:23540/2" value="10k"/>
+<part name="BATTERY_CON_2" library="con-phoenix-254" library_urn="urn:adsk.eagle:library:172" deviceset="MPT4" device="" package3d_urn="urn:adsk.eagle:package:9326/1"/>
 </parts>
 <sheets>
@@
 <instance part="R12" gate="G$1" x="30.48" y="127"/>
 <instance part="SUPPLY5" gate="GND" x="25.4" y="109.22"/>
+<instance part="Q1" gate="G$1" x="45.72" y="17.78" rot="R270"/>
+<instance part="Q2" gate="G$1" x="45.72" y="-7.62" rot="R270"/>
+<instance part="R13" gate="G$1" x="38.1" y="22.86" rot="R90"/>
+<instance part="R14" gate="G$1" x="53.34" y="22.86" rot="R90"/>
+<instance part="R15" gate="G$1" x="38.1" y="-2.54" rot="R90"/>
+<instance part="R16" gate="G$1" x="53.34" y="-2.54" rot="R90"/>
+<instance part="BATTERY_CON_2" gate="-1" x="119.38" y="124.46"/>
+<instance part="BATTERY_CON_2" gate="-2" x="119.38" y="119.38"/>
+<instance part="BATTERY_CON_2" gate="-3" x="119.38" y="114.3"/>
+<instance part="BATTERY_CON_2" gate="-4" x="119.38" y="109.22"/>
 </instances>
 <busses>
@@
 <label x="40.64" y="43.18" size="1.778" layer="95"/>
 </segment>
+<segment>
+<pinref part="R16" gate="G$1" pin="2"/>
+<wire x1="53.34" y1="2.54" x2="53.34" y2="7.62" width="0.1524" layer="91"/>
+<label x="53.34" y="2.54" size="1.778" layer="95" rot="R90"/>
+</segment>
+<segment>
+<pinref part="R14" gate="G$1" pin="2"/>
+<wire x1="53.34" y1="27.94" x2="53.34" y2="33.02" width="0.1524" layer="91"/>
+<label x="53.34" y="27.94" size="1.778" layer="95" rot="R90"/>
+</segment>
 </net>
 <net name="N$1" class="0">
@@
 <label x="-7.62" y="66.04" size="1.778" layer="95"/>
 </segment>
+<segment>
+<pinref part="BATTERY_CON_2" gate="-1" pin="1"/>
+<wire x1="116.84" y1="124.46" x2="111.76" y2="124.46" width="0.1524" layer="91"/>
+<label x="111.76" y="124.46" size="1.778" layer="95"/>
+</segment>
 </net>
 <net name="BATT3" class="0">
@@
 <label x="-7.62" y="60.96" size="1.778" layer="95"/>
 </segment>
+<segment>
+<pinref part="BATTERY_CON_2" gate="-2" pin="1"/>
+<wire x1="116.84" y1="119.38" x2="111.76" y2="119.38" width="0.1524" layer="91"/>
+<label x="111.76" y="119.38" size="1.778" layer="95"/>
+</segment>
 </net>
 <net name="BATT4" class="0">
@@
 <label x="-7.62" y="55.88" size="1.778" layer="95"/>
 </segment>
+<segment>
+<pinref part="BATTERY_CON_2" gate="-3" pin="1"/>
+<wire x1="116.84" y1="114.3" x2="111.76" y2="114.3" width="0.1524" layer="91"/>
+<label x="111.76" y="114.3" size="1.778" layer="95"/>
+</segment>
 </net>
 <net name="BATT5" class="0">
@@
 <label x="43.18" y="55.88" size="1.778" layer="95"/>
 </segment>
+<segment>
+<pinref part="BATTERY_CON_2" gate="-4" pin="1"/>
+<wire x1="116.84" y1="109.22" x2="111.76" y2="109.22" width="0.1524" layer="91"/>
+<label x="111.76" y="109.22" size="1.778" layer="95"/>
+</segment>
 </net>
 <net name="SDA" class="0">
-<segment>
-<pinref part="U$1" gate="G$1" pin="A4"/>
-<wire x1="50.8" y1="60.96" x2="43.18" y2="60.96" width="0.1524" layer="91"/>
-<label x="43.18" y="60.96" size="1.778" layer="95"/>
-</segment>
 <segment>
 <pinref part="MAIN_I2C" gate="-2" pin="S"/>
@@
 <label x="73.66" y="99.06" size="1.778" layer="95"/>
 </segment>
+<segment>
+<pinref part="R15" gate="G$1" pin="1"/>
+<pinref part="Q2" gate="G$1" pin="S"/>
+<wire x1="38.1" y1="-7.62" x2="38.1" y2="-10.16" width="0.1524" layer="91"/>
+<wire x1="38.1" y1="-10.16" x2="40.64" y2="-10.16" width="0.1524" layer="91"/>
+<wire x1="38.1" y1="-10.16" x2="33.02" y2="-10.16" width="0.1524" layer="91"/>
+<junction x="38.1" y="-10.16"/>
+<label x="33.02" y="-10.16" size="1.778" layer="95" rot="MR0"/>
+</segment>
 </net>
 <net name="SCL" class="0">
-<segment>
-<pinref part="U$1" gate="G$1" pin="A5"/>
-<wire x1="50.8" y1="58.42" x2="43.18" y2="58.42" width="0.1524" layer="91"/>
-<label x="43.18" y="58.42" size="1.778" layer="95"/>
-</segment>
 <segment>
 <pinref part="MAIN_I2C" gate="-1" pin="S"/>
 <wire x1="81.28" y1="101.6" x2="73.66" y2="101.6" width="0.1524" layer="91"/>
 <label x="73.66" y="101.6" size="1.778" layer="95"/>
+</segment>
+<segment>
+<pinref part="Q1" gate="G$1" pin="S"/>
+<wire x1="40.64" y1="15.24" x2="38.1" y2="15.24" width="0.1524" layer="91"/>
+<pinref part="R13" gate="G$1" pin="1"/>
+<wire x1="38.1" y1="17.78" x2="38.1" y2="15.24" width="0.1524" layer="91"/>
+<junction x="38.1" y="15.24"/>
+<wire x1="38.1" y1="15.24" x2="33.02" y2="15.24" width="0.1524" layer="91"/>
+<label x="33.02" y="15.24" size="1.778" layer="95" rot="MR0"/>
 </segment>
 </net>
@@
 </segment>
 </net>
+<net name="SDA_HV" class="0">
+<segment>
+<pinref part="U$1" gate="G$1" pin="A4"/>
+<wire x1="50.8" y1="60.96" x2="43.18" y2="60.96" width="0.1524" layer="91"/>
+<label x="43.18" y="60.96" size="1.778" layer="95"/>
+</segment>
+<segment>
+<pinref part="R16" gate="G$1" pin="1"/>
+<wire x1="53.34" y1="-7.62" x2="53.34" y2="-10.16" width="0.1524" layer="91"/>
+<pinref part="Q2" gate="G$1" pin="D"/>
+<wire x1="53.34" y1="-10.16" x2="50.8" y2="-10.16" width="0.1524" layer="91"/>
+<wire x1="53.34" y1="-10.16" x2="58.42" y2="-10.16" width="0.1524" layer="91"/>
+<junction x="53.34" y="-10.16"/>
+<label x="55.88" y="-10.16" size="1.778" layer="95"/>
+</segment>
+</net>
+<net name="SCL_HV" class="0">
+<segment>
+<pinref part="U$1" gate="G$1" pin="A5"/>
+<wire x1="50.8" y1="58.42" x2="43.18" y2="58.42" width="0.1524" layer="91"/>
+<label x="43.18" y="58.42" size="1.778" layer="95"/>
+</segment>
+<segment>
+<pinref part="Q1" gate="G$1" pin="D"/>
+<wire x1="50.8" y1="15.24" x2="53.34" y2="15.24" width="0.1524" layer="91"/>
+<wire x1="53.34" y1="15.24" x2="60.96" y2="15.24" width="0.1524" layer="91"/>
+<pinref part="R14" gate="G$1" pin="1"/>
+<wire x1="53.34" y1="17.78" x2="53.34" y2="15.24" width="0.1524" layer="91"/>
+<junction x="53.34" y="15.24"/>
+<label x="55.88" y="15.24" size="1.778" layer="95"/>
+</segment>
+</net>
+<net name="3.3" class="0">
+<segment>
+<pinref part="U$1" gate="G$1" pin="3.3V"/>
+<wire x1="50.8" y1="76.2" x2="43.18" y2="76.2" width="0.1524" layer="91"/>
+<label x="43.18" y="76.2" size="1.778" layer="95"/>
+</segment>
+<segment>
+<pinref part="Q1" gate="G$1" pin="G"/>
+<pinref part="R13" gate="G$1" pin="2"/>
+<wire x1="43.18" y1="20.32" x2="43.18" y2="27.94" width="0.1524" layer="91"/>
+<wire x1="43.18" y1="27.94" x2="38.1" y2="27.94" width="0.1524" layer="91"/>
+<wire x1="38.1" y1="27.94" x2="38.1" y2="33.02" width="0.1524" layer="91"/>
+<junction x="38.1" y="27.94"/>
+<label x="38.1" y="30.48" size="1.778" layer="95" rot="R90"/>
+</segment>
+<segment>
+<pinref part="R15" gate="G$1" pin="2"/>
+<pinref part="Q2" gate="G$1" pin="G"/>
+<wire x1="38.1" y1="2.54" x2="43.18" y2="2.54" width="0.1524" layer="91"/>
+<wire x1="43.18" y1="2.54" x2="43.18" y2="-5.08" width="0.1524" layer="91"/>
+<wire x1="38.1" y1="2.54" x2="38.1" y2="7.62" width="0.1524" layer="91"/>
+<junction x="38.1" y="2.54"/>
+<label x="38.1" y="2.54" size="1.778" layer="95" rot="R90"/>
+</segment>
+</net>

Commit message: Final commit for battery pcb, added resistor values #2
Parts:
- removed BATTERY_CON_2: (no value), con-phoenix-254:MPT4
- removed R7, R8: (no value), rcl:R-US_R1206
- R1, R4, R5, R6: value (none) -> 10k
- R2: value (none) -> 30k
- R3: value (none) -> 20k
Connections:
- removed net N$4: R7.2, R8.1, U$1.A3
- net BATT2: no longer BATTERY_CON_2-1.1
- net BATT3: no longer BATTERY_CON_2-2.1
- net BATT4: now also U$1.A3; no longer BATTERY_CON_2-3.1, R7.1
- net BATT5: no longer BATTERY_CON_2-4.1, U$1.A6
- net GND: now also MAIN_I2C-3.S; no longer R8.2
Other:
- moved on the sheet: R1, R2, R5, R6
